File: pcb/revA/karabas-pro-revA.kicad_pcb (KiCad board)
At the start: 2 copper layers, 101.6 x 147.3 mm, 129 parts, among them CON1 CF-CARD, CON2 SD, CON3 VGA, CON4 Joystick, CON5 Keyboard, CON6 Mouse, CON7 Audio, CON8 5V DC, J1 Floppy, J2 FPGA JTAG, J3 Floppy 5V, J4 uBus, J5 AVR JTAG, J6 AVR UART, SW1 SW_Push, SW2 SW_Push, U1 EP4CE6E22C8N, U10 ESP-12E, U11 TDA1543, U12 AMS1117-3.3, U13 AMS1117-2.5, U14 AMS1117-1.2, U17 74LS06, U18 74LS38, U2 CY62167EV30, U3 W25Q32JVSS, U4 EPM3128ATC100-5, U5 ATMEGA328-AU, U6 MB8877A, U7 TXB0104PW, U8 TXB0104PW, U9 DS1307Z+, X1 SG-7050CAN, Y1 32768Hz, Y2 16MHz

Commit message: Added pullups
Parts:
- added C45: 470uF, Capacitor_THT:CP_Radial_D12.5mm_P7.50mm, F.Cu at (108.5, 48.0)
- added R38: 10k, Resistor_SMD:R_0805_2012Metric_Pad1.15x1.40mm_HandSolder, B.Cu at (152.7, 87.6)
- added R39: 10k, Resistor_SMD:R_0805_2012Metric_Pad1.15x1.40mm_HandSolder, F.Cu at (148.1, 75.7)
- moved C10 5.84 mm to (113.3, 43.2)
Routing:
- net /~RESET: track 18.6 -> 21.3 mm
- net /SDIR: track 15.8 -> 18.5 mm, vias 0 -> 1

Commit message: Added rev.A documentation
Parts:
- C1, C2: value 100n -> 10uF
- R10, R13, R16: value 1k8 -> 2k
- R12, R15, R18: value 470 -> 510
- R25: value 2k -> 820
- R26, R27: value 270 -> 750
- U3: value W25Q32JVSS -> M25P16
