File: pcb/revB/karabas-pro-revB.sch (KiCad schematic (older format))
At the start: 136 parts, among them CON1 CF-CARD, CON2 SD, CON3 VGA, CON4 Joystick, CON5 Keyboard, CON6 Mouse, CON7 Audio, CON8 5V DC, J1 Floppy, J2 FPGA JTAG, J3 Floppy 5V, J4 uBus, J5 AVR JTAG, J6 AVR UART, SW1 SW_Push, SW2 SW_Push, U1 EP4CE6E22C8N, U10 ESP-12E, U11 TDA1543, U12 AMS1117-3.3, U13 AMS1117-2.5, U14 AMS1117-1.2, U17 74LS06, U18 74LS38, U2 CY62167EV30, U3 M25P16, U4 EPM3128ATC100-5, U5 ATMEGA328-AU, U6 MB8877A, U7 TXB0104PW, U8 TXB0104PW, U9 DS1307Z+, X1 SG-7050CAN, Y1 32768Hz, Y2 16MHz

Commit message: Updated PS/2 footprint
Parts:
- CON5, CON6: footprint footprints:MDIN06SS -> footprints:MINI_DIN_6_33PRIMARY
Changed lines of the file:
@@
 F 0 "CON5" H 12650 3617 50  0000 C CNN
 F 1 "Keyboard" H 12650 3526 50  0000 C CNN
-F 2 "footprints:MDIN06SS" H 12650 3250 50  0001 C CNN
+F 2 "footprints:MINI_DIN_6_33PRIMARY" H 12650 3250 50  0001 C CNN
 F 3 "http://service.powerdynamics.com/ec/Catalog17/Section%2011.pdf" H 12650 3250 50  0001 C CNN
 	1    12650 3250
@@
 F 0 "CON6" H 12650 4617 50  0000 C CNN
 F 1 "Mouse" H 12650 4526 50  0000 C CNN
-F 2 "footprints:MDIN06SS" H 12650 4250 50  0001 C CNN
+F 2 "footprints:MINI_DIN_6_33PRIMARY" H 12650 4250 50  0001 C CNN
 F 3 "http://service.powerdynamics.com/ec/Catalog17/Section%2011.pdf" H 12650 4250 50  0001 C CNN
 	1    12650 4250
@@
 Wire Wire Line
 	4950 10150 5400 10150
+Text Label 4950 10150 0    50   ~ 0
+~LAVR_CS
 Wire Bus Line
 	14200 10200 14200 11000
@@
 Wire Bus Line
 	8750 700  8750 11450
-Text Label 4950 10150 0    50   ~ 0
-~LAVR_CS
 $EndSCHEMATC
