File: pcb/revE/karabas-pro-revE.kicad_pcb (KiCad board)
At the start: 2 copper layers, 101.6 x 147.3 mm, 219 parts, among them CON1 CF-CARD, CON2 SD, CON3 VGA, CON4 Joystick, CON5 Keyboard, CON6 Mouse, CON7 Audio, CON8 12V, CON9 MicroSD', J1 Floppy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

Commit message: Updated rev.E gerbers: added an additional logo on top side
Parts:
- added G***: LOGO, footprints:andy_karpov_logo4_silk, F.Cu at (162.7, 118.2)
