File: pcb/revER/karabas-pro-revER.kicad_sch (KiCad schematic)
At the start: 217 parts, among them CON8 12В, J1 ДИСКОВОД, J10 ВНЕШН. ДЖОЙСТИК, J2 FPGA JTAG, J3 ПИТАНИЕ ДИСКОВОДА, J4 UART2, J5 AVR JTAG, J6 AVR UART, J7 ESP-BUS, J8 МАГН. ВХОД, J9 МАГН. ВЫХОД, Q1 BC856, Q2 BC847, SW4 SW_SPST, U1 EP4CE10E22C8N, U10 ESP-12E, U11 TDA1543, U12 AMS1117-3.3, U13 AMS1117-2.5, U14 AMS1117-1.2, U15 LM2596S-5, U16 LM311, U17 74LS06, U18 74LS38, U19 CY62167EV30LL, U2 CY62167EV30LL, U20 BS62LV1600, U3 W25Q16, U3''1 W25Q16, U4 EPM3128ATC100-10N, U5 ATMEGA328-AU, U6 MB8877A, U7 TXB0104PW, U8 TXB0104PW, U9 DS1307Z+, X1 SG-7050CAN, Y1 32768Hz, Y2 16MHz

Commit message: Updated rev.Ё
Parts:
- added C63: 100n, Capacitor_SMD:C_0805_2012Metric_Pad1.18x1.45mm_HandSolder, symbol Device:C
- added U21: AMS1117-3.3, Package_TO_SOT_SMD:SOT-223-3_TabPin2, symbol Regulator_Linear:AMS1117-3.3
- C13: footprint Capacitor_SMD:C_0805_2012Metric_Pad1.15x1.40mm_HandSolder -> Capacitor_SMD:C_0805_2012Metric_Pad1.18x1.45mm_HandSolder
- CON9: renamed from РАЗЪЕМ9; footprint footprints:MICRO_SD_MOLEX -> footprints:Conn_uSDcard
- renumbered БАТ1 to BT1, КН1 to BTN1, КН2 to BTN2, РАЗЪЕМ1 to CON1, РАЗЪЕМ2 to CON2, РАЗЪЕМ3 to CON3, РАЗЪЕМ4 to CON4, РАЗЪЕМ5 to CON5, РАЗЪЕМ6 to CON6, РАЗЪЕМ7 to CON7
Connections:
- net GND: now also C63.2, U21.1 (GND)
- net VCC: now also C63.1, U21.3 (VI)
- net VCC3_3: no longer C13.1, C54.1, J7.10 (Pin_10), R30.2, R31.2, U10.8 (VCC)
- new net VCC3_3_ESP: C13.1, C54.1, J7.10 (Pin_10), R30.2, R31.2, U10.8 (VCC), U21.2 (VO)
