File: pcb/revF/karabas-pro-revF.kicad_pcb (KiCad board)
At the start: 2 copper layers, 101.6 x 147.3 mm, 232 parts, among them CON1 JOYSTICK, CON2 KEYBOARD, CON3 MOUSE, CON4 12V, CON5 SD CARD, CON6 CF CARD, CON7 SOUND, CON8 VGA, J1 FPGA JTAG, J2 SWD, J3 FDD POWER, J4 FDD, J5 TAPE IN, J6 TAPE OUT, J7 USB C, Q1 IRLML2402, Q2 IRLML2402, Q3 IRLML2402, Q4 IRLML2402, Q5 BC856, SW1 SW_SPST, U1 EP4CE22E22C8N, U10 EPM3128ATC100-10N, U11 LM2596S-5, U12 AMS1117-3.3, U13 AMS1117-2.5, U14 AMS1117-1.2, U15 74LS38, U16 74LS06, U17 MB8877A, U18 ESP-12E, U19 AMS1117-3.3, U2 W25Q16, U20 LM311, U21 TDA1543, U3 CY62167EV30LL, U4 24LC08B, U5 W25Q128JVS, U6 DS3231MZ, U7 LM1117MP-3.3, U8 74HC597, U9 RP2040, X1 50 MHz, Y1 12MHz

Commit message: revF routed
Parts:
- removed C77, C78: 10uF, Capacitor_SMD:C_0805_2012Metric_Pad1.15x1.40mm_HandSolder
- removed J2: SWD, Connector_PinHeader_2.54mm:PinHeader_1x03_P2.54mm_Vertical
- added C25: 100n, Capacitor_SMD:C_0805_2012Metric_Pad1.18x1.45mm_HandSolder, B.Cu at (132.5, 44.4)
- added C26: 10uF, Capacitor_SMD:C_0805_2012Metric_Pad1.18x1.45mm_HandSolder, B.Cu at (134.6, 44.4)
- added C28: 100n, Capacitor_SMD:C_0805_2012Metric_Pad1.18x1.45mm_HandSolder, B.Cu at (132.3, 48.5)
- added C29: 47uF, Capacitor_SMD:CP_Elec_5x5.9, F.Cu at (135.7, 39.4)
- added C48: 100n, Capacitor_SMD:C_0805_2012Metric_Pad1.18x1.45mm_HandSolder, B.Cu at (133.4, 37.3)
- added C52: 100n, Capacitor_SMD:C_0805_2012Metric_Pad1.18x1.45mm_HandSolder, B.Cu at (131.3, 37.3)
- added LOGO_ANDY1: Logo_Open_Hardware_Small, footprints:andy_karpov_logo4_silk, F.Cu at (150.4, 128.0)
- added LOGO_BOTTOM1: Logo_Open_Hardware_Small, footprints:karabas_pro_logo4_copper, B.Cu at (155.8, 127.9)
- added LOGO_TOP1: Logo_Open_Hardware_Small, footprints:karabas_pro_logo4_copper, F.Cu at (133.0, 166.5)
- added R90: 100, Resistor_SMD:R_0805_2012Metric_Pad1.20x1.40mm_HandSolder, B.Cu at (129.2, 37.3)
- added TP1: TP1, TestPoint:TestPoint_Pad_D1.0mm, F.Cu at (124.4, 96.2)
- C31: value 100n -> 47uF; footprint Capacitor_SMD:C_0805_2012Metric_Pad1.15x1.40mm_HandSolder -> Capacitor_SMD:CP_Elec_5x5.9; moved to F.Cu
- R26, R27, R28: value 470 -> 1k
- R71: value 820 -> 220k; footprint Resistor_SMD:R_0805_2012Metric_Pad1.15x1.40mm_HandSolder -> Resistor_SMD:R_0805_2012Metric_Pad1.20x1.40mm_HandSolder
- R72: value 750 -> 220k; footprint Resistor_SMD:R_0805_2012Metric_Pad1.15x1.40mm_HandSolder -> Resistor_SMD:R_0805_2012Metric_Pad1.20x1.40mm_HandSolder
- R73: value 750 -> 100; footprint Resistor_SMD:R_0805_2012Metric_Pad1.15x1.40mm_HandSolder -> Resistor_SMD:R_0805_2012Metric_Pad1.20x1.40mm_HandSolder
- U21: value TDA1543 -> UDA1334ATS; footprint Package_DIP:DIP-8_W7.62mm -> Package_SO:SSOP-16_4.4x5.2mm_P0.65mm
- moved BTN1 16.4 mm to (197.3, 100.7)
- moved BTN2 16.1 mm to (197.3, 117.2)
- moved R71 9.80 mm to (137.5, 37.3), turned to -90 degrees
- moved R73 9.33 mm to (135.4, 37.3), turned to 90 degrees
- moved C31 7.58 mm to (129.8, 39.4), turned to 90 degrees
- moved C3 7.29 mm to (191.6, 103.8)
- moved C17 6.48 mm to (188.2, 110.7)
- moved R72 4.87 mm to (127.2, 37.3), turned to -90 degrees
- moved U21 4.63 mm to (131.6, 48.5)
- moved R11 4.57 mm to (119.9, 91.0)
- moved R13 4.57 mm to (191.6, 99.8)
- moved C18 4.56 mm to (188.7, 115.2), turned to -90 degrees
- moved R40 2.87 mm to (129.1, 140.3)
- moved C16 2.25 mm to (179.2, 120.0), turned to -90 degrees
- moved R34 2.15 mm to (125.3, 139.5)
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Connections:
- C31 pad 1: VCC -> Net-(U21-VOUTR)
- C31 pad 2: GND -> Net-(C31-Pad2)
- R28 pad 1: VCC -> VCC3_3
- R71 pad 1: Net-(U21-VREF) -> GND
- R71 pad 2: GND -> Net-(C29-Pad2)
- R72 pad 1: Net-(U21-AOL) -> GND
- R72 pad 2: GND -> Net-(C31-Pad2)
- R73 pad 1: Net-(U21-AOR) -> Net-(C29-Pad2)
- R73 pad 2: GND -> SND_R
- U1 pad 25: unconnected-(U1-CLK3-Pad25) -> Net-(U1-CLK3)
- U21 pad 4: GND -> VCC3_3
- U21 pad 5: VCC -> GND
- U21 pad 6: Net-(U21-AOL) -> GND
- U21 pad 7: Net-(U21-VREF) -> GND
- U21 pad 8: Net-(U21-AOR) -> GND
Routing:
- net NSTATUS: track 1.16 -> 132.6 mm, vias 1 -> 4
- net VCC3_3: track 491.0 -> 620.0 mm, vias 35 -> 45
- net NCONFIG: track 1.37 -> 128.6 mm, vias 1 -> 4
- net CONF_DONE: track 4.63 -> 87.6 mm, vias 1 -> 4
- net PS2_KB_CLK: track 2.37 -> 79.1 mm, vias 0 -> 3
- net PS2_MS_CLK: track 2.37 -> 78.8 mm, vias 0 -> 5
- net +3.3VP: track 0.00 -> 75.9 mm, vias 0 -> 11
- net DCLK: track 73.7 -> 149.5 mm, vias 3 -> 7
- net DATA0: track 87.1 -> 159.0 mm, vias 5 -> 8
- net SD14: track 0.00 -> 71.0 mm, vias 0 -> 4
- net LFDC_STEP: track 0.00 -> 61.6 mm, vias 0 -> 4
- net SD15: track 0.04 -> 56.5 mm, vias 0 -> 2
- net MA3: track 40.8 -> 93.2 mm, vias 1 -> 4
- net PS2_KB_DATA: track 21.1 -> 68.0 mm, vias 0 -> 1
- net PS2_MS_DATA: track 17.3 -> 63.5 mm, vias 0 -> 3
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Other:
- board text added: "© 2025 andykarpov www.karabas.uk"
- board text removed: "EXT JOYSTICK"
- board text removed: "© 2024 andykarpov www.karabas.uk"

Commit message: DRC passed
Routing:
- net Net-(U18-ADC): track 9.69 -> 5.55 mm, vias 1 -> 0
- net VCC3_3: track 620.0 -> 619.1 mm, vias 45 -> 44

Commit message: Updated revF hw and docs
Parts:
- added JP3: VBUS, Connector_PinHeader_2.54mm:PinHeader_1x02_P2.54mm_Vertical, F.Cu at (197.5, 134.7)
- added TP2: A0, TestPoint:TestPoint_Pad_D1.0mm, F.Cu at (190.1, 115.6)
- added TP3: A1, TestPoint:TestPoint_Pad_D1.0mm, F.Cu at (191.6, 115.6)
- added TP4: A2, TestPoint:TestPoint_Pad_D1.0mm, F.Cu at (192.5, 114.4)
- added TP5: A3, TestPoint:TestPoint_Pad_D1.0mm, F.Cu at (190.2, 113.6)
- C20, C21, C23, C24, C27, C30, C32, C33, C35, C36, C38, C39, C40, C41, C42, C43, C44, C45, C47, C49, C51, C53, C54, C55, C56, C57, C59, C60, C61, C62, C63, C64, C65, C66, C67, C69: footprint Capacitor_SMD:C_0805_2012Metric_Pad1.15x1.40mm_HandSolder -> Capacitor_SMD:C_0805_2012Metric_Pad1.18x1.45mm_HandSolder
- R36, R37: value 470 -> 1k
- moved C59 0.05 mm to (128.8, 93.7)
Connections:
- U9 pad 38: unconnected-(U9-GPIO26_ADC0-Pad38) -> Net-(U9-GPIO26_ADC0)
- U9 pad 39: unconnected-(U9-GPIO27_ADC1-Pad39) -> Net-(U9-GPIO27_ADC1)
- U9 pad 40: unconnected-(U9-GPIO28_ADC2-Pad40) -> Net-(U9-GPIO28_ADC2)
- U9 pad 41: unconnected-(U9-GPIO29_ADC3-Pad41) -> Net-(U9-GPIO29_ADC3)
Routing:
- net VBUS: track 11.2 -> 34.5 mm
- net GND: track 260.3 -> 269.0 mm, vias 263 -> 266
- net Net-(U9-GPIO28_ADC2): track 0.00 -> 5.26 mm
- net Net-(U9-GPIO27_ADC1): track 0.00 -> 4.69 mm
- net VCC: track 492.2 -> 496.5 mm
- net Net-(U9-GPIO29_ADC3): track 0.00 -> 3.06 mm
- net Net-(U9-GPIO26_ADC0): track 0.00 -> 2.71 mm
- net LED_BUSY: track 31.7 -> 29.3 mm
- net MCU_CS: track 68.3 -> 70.3 mm
- net NCONFIG: track 128.6 -> 130.6 mm
- net MCU_MOSI: track 68.0 -> 69.6 mm
- net CONF_DONE: track 87.6 -> 89.1 mm
- net NSTATUS: track 132.6 -> 134.1 mm
- net RP_RESET: track 21.4 -> 22.7 mm
- net MCU_MISO: track 67.0 -> 67.8 mm
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Other:
- board text removed: "РОЗРОБЛЕНО В УКРАЇНІ"
