File: pcb/revF/karabas-pro-revF.kicad_pcb (KiCad board)
At the start: 2 copper layers, 101.6 x 147.3 mm, 245 parts, among them CON1 JOYSTICK, CON2 KEYBOARD, CON3 MOUSE, CON4 12V, CON5 SD CARD, CON6 CF CARD, CON7 SOUND, CON8 VGA, J1 FPGA JTAG, J3 FDD POWER, J4 FDD, J5 TAPE IN, J6 TAPE OUT, J7 USB C, Q1 IRLML2402, Q2 IRLML2402, Q3 IRLML2402, Q4 IRLML2402, Q5 BC856, SW1 SW_SPST, U1 EP4CE22E22C8N, U10 EPM3128ATC100-10N, U11 LM2596S-5, U12 AMS1117-3.3, U13 AMS1117-2.5, U14 AMS1117-1.2, U15 74LS38, U16 74LS06, U17 MB8877A, U18 ESP-12E, U19 AMS1117-3.3, U2 W25Q16, U20 LM311, U21 UDA1334ATS, U3 CY62167EV30LL, U4 24LC08B, U5 W25Q128JVS, U6 DS3231MZ, U7 LM1117MP-3.3, U8 74HC597, U9 RP2040, X1 50 MHz, Y1 12MHz

Commit message: Updated revF
Parts:
- C26, C37, C46, C58: value 10uF -> 10u
- C27: value 1uF -> 1u
- C29, C31: value 47uF -> 47u
- C34: value 470uF -> 470u
- C50: value 220uF -> 220u
- C6, C7: value 22pF -> 22p
- C72: value 100uF -> 100u
- CON1: footprint Connector_Dsub:DSUB-9_Male_Horizontal_P2.77x2.84mm_EdgePinOffset7.70mm_Housed_MountingHolesOffset9.12mm -> Connector_Dsub:DSUB-9_Pins_Horizontal_P2.77x2.84mm_EdgePinOffset7.70mm_Housed_MountingHolesOffset9.12mm
- CON8: footprint Connector_Dsub:DSUB-15-HD_Female_Horizontal_P2.29x1.98mm_EdgePinOffset3.03mm_Housed_MountingHolesOffset4.94mm -> Connector_Dsub:DSUB-15-HD_Socket_Horizontal_P2.29x1.90mm_EdgePinOffset3.03mm_Housed_MountingHolesOffset4.94mm
- D5: footprint Diode_SMD:D_SMB -> Diode_SMD:D_SMB_Handsoldering
- D8, Q1, Q2, Q3, Q4, Q5: footprint Package_TO_SOT_SMD:SOT-23 -> Package_TO_SOT_SMD:SOT-23_Handsoldering
- F1, F2: footprint Fuse:Fuse_1812_4532Metric_Castellated -> Fuse:Fuse_1812_4532Metric_Pad1.30x3.40mm_HandSolder
- R1, R10, R11, R2, R22, R23, R24, R25, R26, R27, R28, R29, R3, R30, R31, R32, R34, R35, R36, R37, R38, R39, R40, R41, R42, R43, R44, R45, R46, R47, R48, R49, R5, R50, R51, R52, R53, R54, R56, R57, R58, R59, R6, R60, R61, R63, R7, R78, R79, R8, R80, R81, R82, R83, R84, R85, R86, R87, R9: footprint Resistor_SMD:R_0805_2012Metric_Pad1.15x1.40mm_HandSolder -> Resistor_SMD:R_0805_2012Metric_Pad1.20x1.40mm_HandSolder
- R33: value 300 -> 330; footprint Resistor_SMD:R_0805_2012Metric_Pad1.15x1.40mm_HandSolder -> Resistor_SMD:R_0805_2012Metric_Pad1.20x1.40mm_HandSolder
- R69: value 33 -> 27; footprint Resistor_SMD:R_0805_2012Metric_Pad1.15x1.40mm_HandSolder -> Resistor_SMD:R_0805_2012Metric_Pad1.20x1.40mm_HandSolder
- R88, R89: value 75 -> 100; footprint Resistor_SMD:R_0805_2012Metric_Pad1.15x1.40mm_HandSolder -> Resistor_SMD:R_0805_2012Metric_Pad1.20x1.40mm_HandSolder
- SW1: footprint Button_Switch_THT:SW_CuK_OS102011MA1QN1_SPDT_Angled -> Button_Switch_THT:SW_Slide_SPDT_Angled_CK_OS102011MA1Q
- U5: footprint Package_SO:SOIC-8_5.23x5.23mm_P1.27mm -> footprints:SOIC-8_5.23x5.23mm_P1.27mm-LONG
- U9: footprint RP2040_minimal:RP2040-QFN-56 -> footprints:QFN-56-1EP_7x7mm_P0.4mm_EP3.2x3.2mm_ThermalViaBig
- X1: footprint Oscillator:Oscillator_SMD_SeikoEpson_SG8002CA-4Pin_7.0x5.0mm -> Oscillator:Oscillator_SMD_SeikoEpson_SG8002CA-4Pin_7.0x5.0mm_HandSoldering
- moved U11 1.92 mm to (118.3, 47.6)
- moved D5 0.97 mm to (107.9, 51.8)
- moved U12 0.80 mm to (113.8, 67.0)
- moved X1 0.54 mm to (117.1, 96.5)
- moved Q1 0.50 mm to (165.5, 74.6)
- moved Q2 0.49 mm to (175.2, 74.7)
- moved Q4 0.46 mm to (175.2, 78.9)
- moved Q3 0.44 mm to (165.5, 78.9)
Routing:
- net VCC3_3: track 618.9 -> 610.4 mm
- net +3.3VP: track 75.5 -> 71.6 mm
- net QSPI_D2: track 14.7 -> 17.1 mm
- net TAPE_OUT: track 162.4 -> 161.2 mm
- net Net-(Q3-D): track 88.4 -> 87.4 mm
- net I2C_SCL: track 20.4 -> 19.6 mm
- net CONF_DONE: track 89.1 -> 88.4 mm
- net Net-(U9-XIN): track 20.8 -> 20.0 mm
- net Net-(C7-Pad1): track 5.75 -> 5.03 mm
- net JOY_L_P9: track 18.7 -> 18.0 mm
- net /interfaces/B: track 22.3 -> 21.6 mm
- net Net-(U21-VOUTR): track 4.24 -> 3.57 mm
- net TMS: track 104.1 -> 103.5 mm
- net VCC: track 496.5 -> 495.9 mm
- net QSPI_D1: track 19.6 -> 20.1 mm
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