File: pcb/revF/karabas-pro-revF.kicad_pcb (KiCad board)
At the start: 2 copper layers, 101.6 x 147.3 mm, 240 parts, among them CON1 JOYSTICK, CON2 KEYBOARD, CON3 MOUSE, CON4 12V, CON5 SD CARD, CON6 CF CARD, CON7 SOUND, CON8 VGA, J1 FPGA JTAG, J2 I2C, J3 FDD POWER, J4 FDD, J5 TAPE IN, J6 TAPE OUT, J7 USB C, Q1 IRLML2402, Q2 IRLML2402, Q3 IRLML2402, Q4 IRLML2402, Q5 BC856, SW1 SW_SPST, U1 EP4CE22E22C8N, U10 EPM3128ATC100-10N, U11 LM2596S-5, U12 AMS1117-3.3, U13 AMS1117-2.5, U14 AMS1117-1.2, U15 74LS38, U16 74LS06, U17 MB8877A, U18 ESP-12E, U19 AMS1117-3.3, U20 LM311, U21 UDA1334ATS, U22 SN74LV1T34DBV, U3 CY62167EV30LL, U4 24LC08B, U5 W25Q128JVS, U6 DS3231MZ, U7 LM1117MP-3.3, U8 74HC597, U9 RP2040, X1 50 MHz, Y1 12MHz

Commit message: minor pcb revF fixes
Routing:
- net RP_RESET: track 23.4 -> 22.7 mm
- net GND: track 205.1 -> 205.7 mm
Changed lines of the file:
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@@
 	)
 	(segment
-		(start 199.0228 113.5674)
-		(end 197.4402 115.15)
-		(width 0.2)
-		(layer "F.Cu")
-		(net 1)
-	)
-	(segment
 		(start 159.568 85.797)
 		(end 159.568 88.773)
@@
 	)
 	(segment
-		(start 194.204 115.646)
-		(end 194.204 117.254)
+		(start 194.204 118.304)
+		(end 194.205 118.305)
 		(width 0.2)
 		(layer "F.Cu")
@@
 	)
 	(segment
-		(start 196.794364 115.15)
-		(end 196.664364 115.28)
-		(width 0.2)
-		(layer "F.Cu")
-		(net 1)
-	)
-	(segment
 		(start 157.808692 100.02199)
 		(end 157.818 100.031298)
@@
 	)
 	(segment
+		(start 199.0228 113.5674)
+		(end 197.3102 115.28)
+		(width 0.2)
+		(layer "F.Cu")
+		(net 1)
+	)
+	(segment
 		(start 158.04201 100.02199)
 		(end 159.004 99.06)
@@
 	)
 	(segment
+		(start 194.57 115.28)
+		(end 194.204 115.646)
+		(width 0.2)
+		(layer "F.Cu")
+		(net 1)
+	)
+	(segment
 		(start 160.568 101.147)
 		(end 160.568 99.382501)
@@
 	)
 	(segment
-		(start 196.664364 115.28)
-		(end 194.57 115.28)
-		(width 0.2)
-		(layer "F.Cu")
-		(net 1)
-	)
-	(segment
 		(start 162.663341 98.204343)
 		(end 162.663341 97.178659)
@@
 	)
 	(segment
-		(start 194.204 117.254)
+		(start 194.205 118.305)
 		(end 195.255 118.305)
 		(width 0.2)
@@
 	)
 	(segment
-		(start 197.4402 115.15)
-		(end 196.794364 115.15)
+		(start 194.204 115.646)
+		(end 194.204 118.304)
 		(width 0.2)
 		(layer "F.Cu")
@@
 	)
 	(segment
+		(start 197.3102 115.28)
+		(end 194.57 115.28)
+		(width 0.2)
+		(layer "F.Cu")
+		(net 1)
+	)
+	(segment
 		(start 129.7468 117.4672)
 		(end 128.7272 117.4672)
@@
 	)
 	(segment
-		(start 194.57 115.28)
-		(end 194.204 115.646)
-		(width 0.2)
-		(layer "F.Cu")
-		(net 1)
-	)
-	(segment
 		(start 129.7468 107.9672)
 		(end 130.572813 107.9672)
@@
 	)
 	(segment
-		(start 197.53995 115.55)
-		(end 197.95 115.96005)
+		(start 185.9923 121.3179)
+		(end 186.0644 121.39)
 		(width 0.2)
 		(layer "F.Cu")
@@
 	)
 	(segment
-		(start 195.255 116.155)
-		(end 196.55 116.155)
+		(start 197.95 116.155)
+		(end 199.405 116.155)
 		(width 0.2)
 		(layer "F.Cu")
@@
 	)
 	(segment
-		(start 185.9923 121.3179)
-		(end 186.0644 121.39)
+		(start 196.73995 116.15)
+		(end 197.945 116.15)
 		(width 0.2)
 		(layer "F.Cu")
@@
 	)
 	(segment
-		(start 196.96005 115.55)
-		(end 197.53995 115.55)
+		(start 197.945 116.15)
+		(end 197.95 116.155)
 		(width 0.2)
 		(layer "F.Cu")
@@
 	)
 	(segment
-		(start 197.95 116.155)
-		(end 199.405 116.155)
+		(start 196.73495 116.155)
+		(end 196.73995 116.15)
 		(width 0.2)
 		(layer "F.Cu")
@@
 	)
 	(segment
-		(start 197.95 115.96005)
-		(end 197.95 116.155)
-		(width 0.2)
-		(layer "F.Cu")
-		(net 20)
-	)
-	(segment
 		(start 185.9923 120.5409)
 		(end 185.9923 121.3179)
@@
 	)
 	(segment
-		(start 196.55 115.96005)
-		(end 196.96005 115.55)
+		(start 186.0644 121.39)
+		(end 186.0644 121.65)
 		(width 0.2)
 		(layer "F.Cu")
@@
 	)
 	(segment
-		(start 186.0644 121.39)
-		(end 186.0644 121.65)
+		(start 195.255 116.155)
+		(end 196.73495 116.155)
 		(width 0.2)
 		(layer "F.Cu")
@@
 		(width 0.2)
 		(layer "F.Cu")
-		(net 20)
-	)
-	(segment
-		(start 196.55 116.155)
-		(end 196.55 115.96005)
-		(width 0.2)
-		(layer "F.Cu")

Commit message: PCB revF a4
Parts:
- removed R71, R72: 220k, Resistor_SMD:R_0805_2012Metric_Pad1.20x1.40mm_HandSolder
- removed R73, R90: 100, Resistor_SMD:R_0805_2012Metric_Pad1.20x1.40mm_HandSolder
- removed TP3: A1, TestPoint:TestPoint_Pad_D1.0mm
- removed TP4: A2, TestPoint:TestPoint_Pad_D1.0mm
- removed TP5: A3, TestPoint:TestPoint_Pad_D1.0mm
- removed U6: DS3231MZ, Package_SO:SOIC-8_3.9x4.9mm_P1.27mm
- added C75: 10u, Capacitor_SMD:C_0805_2012Metric_Pad1.18x1.45mm_HandSolder, F.Cu at (134.0, 37.9)
- added C77: 100n, Capacitor_SMD:C_0805_2012Metric_Pad1.18x1.45mm_HandSolder, F.Cu at (134.0, 40.0)
- added C78: 10u, Capacitor_SMD:C_0805_2012Metric_Pad1.18x1.45mm_HandSolder, B.Cu at (129.2, 48.9)
- added C79: 100n, Capacitor_SMD:C_0805_2012Metric_Pad1.18x1.45mm_HandSolder, B.Cu at (127.0, 48.8)
- added R4: 10k, Resistor_SMD:R_0805_2012Metric_Pad1.20x1.40mm_HandSolder, F.Cu at (130.4, 41.0)
- added R5: 10k, Resistor_SMD:R_0805_2012Metric_Pad1.20x1.40mm_HandSolder, F.Cu at (128.3, 41.0)
- added R7: 1k, Resistor_SMD:R_0805_2012Metric_Pad1.20x1.40mm_HandSolder, B.Cu at (132.2, 49.8)
- added U2: DS1307Z+, Package_SO:SOIC-8_3.9x4.9mm_P1.27mm, F.Cu at (183.8, 135.3)
- added Y2: 32768, Crystal:Crystal_C26-LF_D2.1mm_L6.5mm_Horizontal_1EP_style2, F.Cu at (182.7, 141.6)
- C25: moved to F.Cu
- C29: value 47u -> 10u; footprint Capacitor_SMD:CP_Elec_5x5.9 -> Capacitor_SMD:C_0805_2012Metric_Pad1.18x1.45mm_HandSolder; moved to B.Cu
- C31: value 47u -> 2n2; footprint Capacitor_SMD:CP_Elec_5x5.9 -> Capacitor_SMD:C_0805_2012Metric_Pad1.18x1.45mm_HandSolder; moved to B.Cu
- C48: value 100n -> 2n2
- C52: value 100n -> 2u2; moved to F.Cu
- U21: value UDA1334ATS -> PCM5102A; footprint footprints:SSOP-16_4.4x5.2mm_P0.65mm-extended -> Package_SO:TSSOP-20_4.4x6.5mm_P0.65mm
- moved C2 12.1 mm to (190.4, 135.3)
- moved C26 8.56 mm to (130.4, 37.0), turned to -90 degrees
- moved C29 7.75 mm to (128.3, 37.0), turned to -90 degrees
- moved C48 6.32 mm to (128.3, 41.1), turned to 90 degrees
- moved C52 5.53 mm to (134.0, 42.1), turned to 0 degrees
- moved C25 3.88 mm to (136.1, 45.9)
- moved R15 2.43 mm to (185.5, 137.3)
- moved R14 2.31 mm to (185.5, 135.1)
- moved C31 1.83 mm to (130.4, 41.1)
- moved C18 1.22 mm to (187.5, 115.0)
- moved BT1 1.13 mm to (172.7, 146.8)
- moved C28 0.91 mm to (132.3, 47.6)
- moved U21 0.79 mm to (131.1, 47.9), turned to -90 degrees
Connections:
- net Net-(U18-~{RST}) renamed ~{ESP_RESET}
- C2 pad 1: VCC3_3 -> VCC
- C25 pad 1: Net-(U21-Vref(DAC)) -> VCC3_3
- C26 pad 1: Net-(U21-Vref(DAC)) -> SND_L
- C26 pad 2: GND -> Net-(C26-Pad2)
- C29 pad 1: Net-(U21-VOUTL) -> SND_R
- C31 pad 1: Net-(U21-VOUTR) -> GND
- C31 pad 2: Net-(C31-Pad2) -> Net-(C26-Pad2)
- C48 pad 1: SND_R -> GND
- C48 pad 2: GND -> Net-(C29-Pad2)
- C52 pad 1: SND_L -> Net-(U21-CAPM)
- C52 pad 2: GND -> Net-(U21-CAPP)
- U18 pad 18: unconnected-(U18-GPIO0-Pad18) -> ~{ESP_BOOT}
- U21 pad 1: LSND_BS -> VCC3_3
- U21 pad 12: Net-(U21-Vref(DAC)) -> GND
- U21 pad 13: VCC3_3 -> LSND_BS
- U21 pad 14: Net-(U21-VOUTL) -> LSND_DAT
- U21 pad 15: GND -> LSND_WS
- U21 pad 16: Net-(U21-VOUTR) -> GND
- U21 pad 2: LSND_WS -> Net-(U21-CAPP)
- U21 pad 3: LSND_DAT -> GND
- U21 pad 4: VCC3_3 -> Net-(U21-CAPM)
- U21 pad 5: GND -> Net-(U21-VNEG)
- U21 pad 6: GND -> Net-(U21-OUTL)
- U21 pad 7: GND -> Net-(U21-OUTR)
- U21 pad 8: GND -> VCC3_3
- U9 pad 39: Net-(U9-GPIO27_ADC1) -> unconnected-(U9-GPIO27_ADC1-Pad39)
- U9 pad 40: Net-(U9-GPIO28_ADC2) -> unconnected-(U9-GPIO28_ADC2-Pad40)
- U9 pad 41: Net-(U9-GPIO29_ADC3) -> unconnected-(U9-GPIO29_ADC3-Pad41)
Routing:
- net SND_L: track 19.9 -> 9.25 mm
- net Net-(U2-X1): track 0.00 -> 10.0 mm
- net VCC: track 511.0 -> 520.3 mm
- net Net-(U21-LDOO): track 0.00 -> 8.30 mm, vias 0 -> 1
- net Net-(U21-VNEG): track 0.00 -> 7.77 mm
- net Net-(U21-VOUTL): track 7.52 -> 0.00 mm
- net SND_R: track 12.1 -> 4.68 mm
- net VCC3_3: track 684.9 -> 691.2 mm, vias 47 -> 46
- net Net-(U2-X2): track 0.00 -> 6.15 mm
- net Net-(U21-Vref(DAC)): track 5.48 -> 0.00 mm, vias 1 -> 0
- net Net-(U9-GPIO28_ADC2): track 5.26 -> 0.00 mm
- net I2C_SDA: track 121.4 -> 125.7 mm, vias 3 -> 5
- net Net-(U9-GPIO27_ADC1): track 4.04 -> 0.00 mm
- net Net-(U21-OUTR): track 0.00 -> 3.81 mm
- net Net-(U21-VOUTR): track 3.57 -> 0.00 mm
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Other:
- board text added: "© 2026 andykarpov www.karabas.uk"
- board text removed: "© 2025 andykarpov www.karabas.uk"
