File: pcb/revF/fpga.kicad_sch (KiCad schematic)
At the start: 19 parts, among them J2 FPGA JTAG, U1 EP4CE10E22C8N, U3 W25Q16, U3''1 W25Q16, X1 50 MHz

Commit message: New schematics / revF
Parts:
- removed JP2: FLASH 1/2, Connector_PinHeader_2.54mm:PinHeader_1x03_P2.54mm_Vertical, symbol Jumper:Jumper_3_Bridged12
- removed R57: 27, Resistor_SMD:R_0805_2012Metric_Pad1.15x1.40mm_HandSolder, symbol Device:R
- removed R58, R60: 10k, Resistor_SMD:R_0805_2012Metric_Pad1.15x1.40mm_HandSolder, symbol Device:R
- removed U3''1: W25Q16, footprints:SOIC-8_5.23x5.23mm_P1.27mm-LONG, symbol Memory_Flash:W25Q32JVSS
- added JP2: Flashboot, symbol Jumper:Jumper_2_Open
- added R85: 10k, Resistor_SMD:R_0805_2012Metric_Pad1.15x1.40mm_HandSolder, symbol Device:R
- U1: value EP4CE10E22C8N -> EP4CE22E22C8N; symbol retro:EP4CE6E22C8N -> retro:EP4CE22E22C8N
Connections:
- net BEEPER is gone; now on net SD13: U1.86 (IO(DEV_OE))
- net NCSO1 is gone; now on net NCSO: R59.1, U3.1 (~{CS})
- net UART2_CTS is gone; now on net VCC1_2: U1.138 (VCCINT)
- net UART2_TX is gone; now on net SD14: U1.141 (IO)
- net UART_CTS is gone; now on net VCC2_5: U1.3 (VCCA3)
- net UART_RX is gone; now on net GND: U1.2 (GNDA3)
- net UART_TX is gone; now on net VCC1_2: U1.1 (VCCD_PLL3)
- net ~{MRD} is gone; now on net VCC1_2: U1.34 (VCCINT)
- net ~{RAMCE1} is gone; now on net MD4: U1.121 (IO)
- net ~{RAMCE2} is gone; now on net MA3: U1.120 (IO)
- net ~{RAMCE3} is gone; now on net SD15: U1.7 (IO)
- net ~{SD_DET} is gone; now on net SD8: U1.91 (CLK4)
- net GND: now also U1.74 (GNDA4), JP2.2 (B); no longer U1.94 (MSEL0)
- net MA3: no longer U1.70 (IO)
- net MD4: no longer U1.38 (IO)
- net SD13: no longer U1.75 (IO)
- net SD14: no longer U1.74 (IO)
- net SD15: no longer U1.73 (IO)
- net SD8: no longer U1.84 (IO)
- net VCC1_2: now also U1.38 (VCCINT), U1.70 (VCCINT), U1.73 (VCCD_PLL4), U1.84 (VCCINT)
- net VCC2_5: now also U1.75 (VCCA4)
- net VCC3_3: now also R85.2
- net LAVR_MISO renamed MCU_MISO
- net LAVR_MOSI renamed MCU_MOSI
- net LAVR_SCK renamed MCU_SCK
- net UART2_RX: no longer names the net of U1.25 (CLK3)
- net ~{LAVR_CS} renamed MCU_CS
- new net MSEL0: JP2.1 (A), R85.1, U1.94 (MSEL0)
- no-connect marks 3 -> 4
Other:
- note added: "Clock"
- note added: "Optional conf flash"
- note removed: "Conf Flash"
- note removed: "Flash Selector"
- moved on the sheet: J2, R1, R2, R3, R59, R77, X1

Commit message: revF wip
Parts:
- JP1: renamed from JP2; footprint (none) -> Connector_PinHeader_2.54mm:PinHeader_1x02_P2.54mm_Vertical
- R4: renamed from R85; footprint Resistor_SMD:R_0805_2012Metric_Pad1.15x1.40mm_HandSolder -> Resistor_SMD:R_0805_2012Metric_Pad1.20x1.40mm_HandSolder
- renumbered J2 to J1, R33 to R1, R3 to R10, R77 to R11, R34 to R2, R35 to R3, R59 to R5, R1 to R6, R4 to R7, R5 to R8, R2 to R9, U3 to U2
Other:
- note added: "U1 can be one of the following: EP4CE6 EP4CE10 EP4CE15 EP4CE22 EP3C5 EP3C10 EP3C15 EP3C25"

Commit message: revF routed
Parts:
- added TP1: TP1, TestPoint:TestPoint_Pad_D1.0mm, symbol Connector:TestPoint
Connections:
- net at U1.25 (CLK3): now also TP1.1
- no-connect marks 4 -> 3
Other:
- note added: "Pin changes comparing to the previos revE: - UART_TX,RX,CTS moved to the MCU side - UART2_TX,RX,CTS was removed - RAMCE3,RAMCE2,RAMCE1,MRD was removed - BEEPER removed - SD_DET removed - MD4 -> pin_21 - MA3 -> pin_20 - SD15 -> pin_7 - SD14 -> pin_141 - SD13 -> pin_86 - SD8 -> pin_91"

Commit message: Updated revF hw and docs
Parts:
- TP1: now left out of the parts list
- U2: now not fitted; now left out of the parts list
Changed lines of the file:
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@@
 		(unit 1)
 		(exclude_from_sim no)
-		(in_bom yes)
+		(in_bom no)
 		(on_board yes)
 		(dnp no)
@@
 		(unit 1)
 		(exclude_from_sim no)
-		(in_bom yes)
-		(on_board yes)
-		(dnp no)
+		(in_bom no)
+		(on_board yes)
+		(dnp yes)
 		(property "Reference" "U2"
 			(at 231.14 25.6286 0)

Commit message: Updated revF
Parts:
- R1, R10, R11, R2, R3, R5, R6, R7, R8, R9: footprint Resistor_SMD:R_0805_2012Metric_Pad1.15x1.40mm_HandSolder -> Resistor_SMD:R_0805_2012Metric_Pad1.20x1.40mm_HandSolder
- X1: footprint Oscillator:Oscillator_SMD_SeikoEpson_SG8002CA-4Pin_7.0x5.0mm -> Oscillator:Oscillator_SMD_SeikoEpson_SG8002CA-4Pin_7.0x5.0mm_HandSoldering
Changed lines of the file:
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@@
 			)
 		)
-		(property "Footprint" "Resistor_SMD:R_0805_2012Metric_Pad1.15x1.40mm_HandSolder"
+		(property "Footprint" "Resistor_SMD:R_0805_2012Metric_Pad1.20x1.40mm_HandSolder"
 			(at 137.16 188.468 90)
 			(effects
@@
 			)
 		)
-		(property "Footprint" "Resistor_SMD:R_0805_2012Metric_Pad1.15x1.40mm_HandSolder"
+		(property "Footprint" "Resistor_SMD:R_0805_2012Metric_Pad1.20x1.40mm_HandSolder"
 			(at 239.522 91.44 90)
 			(effects
@@
 			)
 		)
-		(property "Footprint" "Resistor_SMD:R_0805_2012Metric_Pad1.15x1.40mm_HandSolder"
+		(property "Footprint" "Resistor_SMD:R_0805_2012Metric_Pad1.20x1.40mm_HandSolder"
 			(at 137.16 173.228 90)
 			(effects
@@
 			)
 		)
-		(property "Footprint" "Resistor_SMD:R_0805_2012Metric_Pad1.15x1.40mm_HandSolder"
+		(property "Footprint" "Resistor_SMD:R_0805_2012Metric_Pad1.20x1.40mm_HandSolder"
 			(at 248.92 124.968 90)
 			(effects
@@
 			)
 		)
-		(property "Footprint" "Oscillator:Oscillator_SMD_SeikoEpson_SG8002CA-4Pin_7.0x5.0mm"
+		(property "Footprint" "Oscillator:Oscillator_SMD_SeikoEpson_SG8002CA-4Pin_7.0x5.0mm_HandSoldering"
 			(at 255.27 132.08 0)
 			(effects
@@
 			)
 		)
-		(property "Footprint" "Resistor_SMD:R_0805_2012Metric_Pad1.15x1.40mm_HandSolder"
+		(property "Footprint" "Resistor_SMD:R_0805_2012Metric_Pad1.20x1.40mm_HandSolder"
 			(at 207.01 29.718 90)
 			(effects
@@
 			)
 		)
-		(property "Footprint" "Resistor_SMD:R_0805_2012Metric_Pad1.15x1.40mm_HandSolder"
+		(property "Footprint" "Resistor_SMD:R_0805_2012Metric_Pad1.20x1.40mm_HandSolder"
 			(at 137.16 180.848 90)
 			(effects
@@
 			)
 		)
-		(property "Footprint" "Resistor_SMD:R_0805_2012Metric_Pad1.15x1.40mm_HandSolder"
+		(property "Footprint" "Resistor_SMD:R_0805_2012Metric_Pad1.20x1.40mm_HandSolder"
 			(at 243.84 36.068 90)
 			(effects
@@
 			)
 		)
-		(property "Footprint" "Resistor_SMD:R_0805_2012Metric_Pad1.15x1.40mm_HandSolder"
+		(property "Footprint" "Resistor_SMD:R_0805_2012Metric_Pad1.20x1.40mm_HandSolder"
 			(at 247.142 91.44 90)
 			(effects
@@
 			)
 		)
-		(property "Footprint" "Resistor_SMD:R_0805_2012Metric_Pad1.15x1.40mm_HandSolder"
+		(property "Footprint" "Resistor_SMD:R_0805_2012Metric_Pad1.20x1.40mm_HandSolder"
 			(at 243.84 43.688 90)
 			(effects
@@
 			)
 		)
-		(property "Footprint" "Resistor_SMD:R_0805_2012Metric_Pad1.15x1.40mm_HandSolder"
+		(property "Footprint" "Resistor_SMD:R_0805_2012Metric_Pad1.20x1.40mm_HandSolder"
 			(at 243.332 69.85 90)
 			(effects

Commit message: RevF pcb
Parts:
- JP1: now not fitted; now left out of the parts list
Connections:
- net TP1: now reaches TP1.1, U1.25 (CLK3)
Other:
- note added: "Pin changes comparing to the previos revE: - UART_TX,RX,CTS moved to the MCU side - UART2_TX,RX,CTS was removed - RAMCE3,RAMCE2,RAMCE1,MRD was removed - BEEPER removed - SD_DET removed - MD4 -> pin_121 - MA3 -> pin_120 - SD15 -> pin_7 - SD14 -> pin_141 - SD13 -> pin_86 - SD8 -> pin_91"
- note removed: "Pin changes comparing to the previos revE: - UART_TX,RX,CTS moved to the MCU side - UART2_TX,RX,CTS was removed - RAMCE3,RAMCE2,RAMCE1,MRD was removed - BEEPER removed - SD_DET removed - MD4 -> pin_21 - MA3 -> pin_20 - SD15 -> pin_7 - SD14 -> pin_141 - SD13 -> pin_86 - SD8 -> pin_91"
- moved on the sheet: TP1
Changed lines of the file:
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@@
 		)
 	)
-	(text "Pin changes comparing to the previos revE:\n- UART_TX,RX,CTS moved to the MCU side\n- UART2_TX,RX,CTS was removed\n- RAMCE3,RAMCE2,RAMCE1,MRD was removed\n- BEEPER removed\n- SD_DET removed\n- MD4 -> pin_21\n- MA3 -> pin_20\n- SD15 -> pin_7\n- SD14 -> pin_141\n- SD13 -> pin_86\n- SD8 -> pin_91\n"
+	(text "Pin changes comparing to the previos revE:\n- UART_TX,RX,CTS moved to the MCU side\n- UART2_TX,RX,CTS was removed\n- RAMCE3,RAMCE2,RAMCE1,MRD was removed\n- BEEPER removed\n- SD_DET removed\n- MD4 -> pin_121\n- MA3 -> pin_120\n- SD15 -> pin_7\n- SD14 -> pin_141\n- SD13 -> pin_86\n- SD8 -> pin_91\n"
 		(exclude_from_sim no)
 		(at 175.514 144.78 0)
@@
 	)
 	(junction
+		(at 22.86 105.41)
+		(diameter 0)
+		(color 0 0 0 0)
+	)
+	(junction
 		(at 46.99 144.78)
 		(diameter 0)
@@
 	(wire
 		(pts
+			(xy 20.32 105.41) (xy 22.86 105.41)
+		)
+		(stroke
+			(width 0)
+			(type default)
+		)
+	)
+	(wire
+		(pts
 			(xy 140.97 171.45) (xy 143.51 171.45)
 		)
@@
 	(wire
 		(pts
+			(xy 22.86 107.95) (xy 22.86 105.41)
+		)
+		(stroke
+			(width 0)
+			(type default)
+		)
+	)
+	(wire
+		(pts
 			(xy 147.32 74.93) (xy 149.86 74.93)
 		)
@@
 	(wire
 		(pts
+			(xy 21.59 107.95) (xy 22.86 107.95)
+		)
+		(stroke
+			(width 0)
+			(type default)
+		)
+	)
+	(wire
+		(pts
 			(xy 241.3 80.01) (xy 248.92 80.01)
 		)
@@
 	(wire
 		(pts
-			(xy 33.02 105.41) (xy 35.56 105.41)
-		)
-		(stroke
-			(width 0)
-			(type default)
-		)
-	)
-	(wire
-		(pts
 			(xy 100.33 31.75) (xy 100.33 34.29)
 		)
@@
 	(wire
 		(pts
+			(xy 22.86 105.41) (xy 35.56 105.41)
+		)
+		(stroke
+			(width 0)
+			(type default)
+		)
+	)
+	(wire
+		(pts
 			(xy 149.86 62.23) (xy 147.32 62.23)
 		)
@@
 		)
 	)
+	(global_label "TP1"
+		(shape input)
+		(at 20.32 105.41 180)
+		(fields_autoplaced yes)
+		(effects
+			(font
+				(size 1.27 1.27)
+			)
+			(justify right)
+		)
+		(property "Intersheetrefs" "${INTERSHEET_REFS}"
+			(at 14.5419 105.41 0)
+			(effects
+				(font
+					(size 1.27 1.27)
+				)
+				(justify right)
+				(hide yes)
+			)
+		)
+	)
 	(global_label "SD0"
 		(shape input)
@@
 	(symbol
 		(lib_id "Connector:TestPoint")
-		(at 33.02 105.41 90)
+		(at 21.59 107.95 90)
 		(unit 1)
 		(exclude_from_sim no)
@@
 		(dnp no)
 		(property "Reference" "TP1"
-			(at 26.924 105.41 90)
+			(at 15.494 107.95 90)
 			(effects
 				(font
@@
 		)
 		(property "Value" "TP1"
-			(at 29.718 102.87 90)
+			(at 18.288 105.41 90)
 			(effects
 				(font
@@
 		)
 		(property "Footprint" "TestPoint:TestPoint_Pad_D1.0mm"
-			(at 33.02 100.33 0)
+			(at 21.59 102.87 0)
 			(effects
 				(font
@@
 		)
 		(property "Datasheet" "~"
-			(at 33.02 100.33 0)
+			(at 21.59 102.87 0)
 			(effects
 				(font
@@
 		)
 		(property "Description" "test point"
-			(at 33.02 105.41 0)
+			(at 21.59 107.95 0)
 			(effects
 				(font
@@
 		(unit 1)
 		(exclude_from_sim no)
-		(in_bom yes)
+		(in_bom no)
 		(on_board yes)
-		(dnp no)
+		(dnp yes)
 		(fields_autoplaced yes)
 		(property "Reference" "JP1"

Commit message: Refactored revF alpha2
Parts:
- TP1: value TP1 -> CLK3
Connections:
- net TAPE_OUT is gone; now on net ~{SD_CS}: U1.10 (IO)
- net LFDC_STEP: now also U1.55 (CLK12); no longer U1.119 (IO)
- net MA1: now also U1.85 (IO); no longer U1.72 (IO)
- net MA10: now also U1.60 (IO); no longer U1.54 (CLK13)
- net MA11: now also U1.59 (IO); no longer U1.53 (CLK14)
- net MA12: now also U1.58 (IO); no longer U1.52 (CLK15)
- net MA17: now also U1.69 (IO); no longer U1.65 (IO)
- net MA18: now also U1.68 (IO); no longer U1.64 (IO)
- net MA19: now also U1.66 (IO(RUP2)); no longer U1.59 (IO)
- net MA2: now also U1.83 (IO); no longer U1.71 (IO)
- net MA3: now also U1.80 (IO); no longer U1.120 (IO)
- net MA4: now also U1.77 (IO(RDN3)); no longer U1.69 (IO)
- net MA5: now also U1.76 (IO(RUP3)); no longer U1.68 (IO)
- net MA6: now also U1.72 (IO); no longer U1.67 (IO(RDN2))
- net MA7: now also U1.71 (IO); no longer U1.66 (IO(RUP2))
- net MA8: now also U1.65 (IO); no longer U1.58 (IO)
- net MA9: now also U1.64 (IO); no longer U1.55 (CLK12)
- net MCU_CS: now also U1.53 (CLK14); no longer U1.88 (CLK7)
- net MCU_MISO: now also U1.86 (IO(DEV_OE)); no longer U1.87 (IO(DEV_CLRN))
- net MCU_MOSI: now also U1.52 (CLK15); no longer U1.90 (CLK5)
- net MCU_SCK: now also U1.54 (CLK13); no longer U1.89 (CLK6)
- net MD4: now also U1.11 (IO); no longer U1.121 (IO)
- net SD10: now also U1.89 (CLK6); no longer U1.80 (IO)
- net SD11: now also U1.88 (CLK7); no longer U1.77 (IO(RDN3))
- net SD12: now also U1.126 (CLK8); no longer U1.76 (IO(RUP3))
- net SD13: now also U1.127 (CLK9); no longer U1.86 (IO(DEV_OE))
- net SD14: now also U1.128 (CLK10); no longer U1.141 (IO)
- net SD15: now also U1.129 (CLK11); no longer U1.7 (IO)
- net SD7: now also U1.87 (IO(DEV_CLRN)); no longer U1.85 (IO)
- net SD9: now also U1.90 (CLK5); no longer U1.83 (IO)
- net SD_DI: now also U1.7 (IO); no longer U1.115 (IO(RDN4))
- net VCC1_2: now also U1.124 (VCCINT)
- net VGA_B0: now also U1.120 (IO); no longer U1.126 (CLK8)
- net VGA_B1: now also U1.121 (IO); no longer U1.127 (CLK9)
- net VGA_B2: now also U1.125 (IO); no longer U1.128 (CLK10)
- net VGA_G0: now also U1.132 (IO); no longer U1.129 (CLK11)
- net VGA_G1: now also U1.133 (IO); no longer U1.132 (IO)
- net VGA_G2: now also U1.135 (IO); no longer U1.133 (IO)
- net VGA_HS: now also U1.119 (IO); no longer U1.125 (IO)
- net VGA_R0: now also U1.136 (IO); no longer U1.135 (IO)
- net VGA_R1: now also U1.137 (IO); no longer U1.136 (IO)
- net VGA_R2: now also U1.141 (IO); no longer U1.137 (IO)
- net VGA_VS: now also U1.115 (IO(RDN4)); no longer U1.124 (VCCINT)
- net ~{MWR}: now also U1.67 (IO(RDN2)); no longer U1.60 (IO)
- net ~{SD_CS}: no longer U1.11 (IO)
- net TP1: no longer names the net of TP1.1, U1.25 (CLK3)
Other:
- note added: "SD[7:0] - выходы в CPLD SD[15:8] - входы от CPLD CLK, CLK2, NRESET, SA, SDIR - выходы в CPLD CPLD_CLK - 116 (BUS) CPLD_CLK2 - 8 (FDD)"
- note removed: "Pin changes comparing to the previos revE: - UART_TX,RX,CTS moved to the MCU side - UART2_TX,RX,CTS was removed - RAMCE3,RAMCE2,RAMCE1,MRD was removed - BEEPER removed - SD_DET removed - MD4 -> pin_121 - MA3 -> pin_120 - SD15 -> pin_7 - SD14 -> pin_141 - SD13 -> pin_86 - SD8 -> pin_91"
- note removed: "U1 can be one of the following: EP4CE6 EP4CE10 EP4CE15 EP4CE22 EP3C5 EP3C10 EP3C15 EP3C25"
- moved on the sheet: R1, R2, R3

Commit message: PCB RevF a3
Parts:
- removed JP1: Flashboot, Connector_PinHeader_2.54mm:PinHeader_1x02_P2.54mm_Vertical, symbol Jumper:Jumper_2_Open
- removed R4, R5, R8: 10k, Resistor_SMD:R_0805_2012Metric_Pad1.20x1.40mm_HandSolder, symbol Device:R
- removed R7: 27, Resistor_SMD:R_0805_2012Metric_Pad1.20x1.40mm_HandSolder, symbol Device:R
- removed TP1: CLK3, TestPoint:TestPoint_Pad_D1.0mm, symbol Connector:TestPoint
- removed U2: W25Q16, footprints:SOIC-8_5.23x5.23mm_P1.27mm-LONG, symbol Memory_Flash:W25Q32JVSS
Connections:
- net MSEL0 is gone; now on net GND: U1.94 (MSEL0)
- net GND: now also U1.96 (MSEL1)
- net VCC2_5: no longer U1.96 (MSEL1)
- net ~{MCU_SD_CS}: now reaches U1.25 (CLK3)
- net ASDO renamed SD_SCK
- net NCSO renamed TAPE_OUT
Other:
- note removed: "Optional conf flash"
- note removed: "SD[7:0] - выходы в CPLD SD[15:8] - входы от CPLD CLK, CLK2, NRESET, SA, SDIR - выходы в CPLD CPLD_CLK - 116 (BUS) CPLD_CLK2 - 8 (FDD)"
- moved on the sheet: J1, R1, R10, R11, R2, R3, R6, R9, X1
