File: pcb/revF/interfaces.kicad_sch (KiCad schematic)
At the start: 49 parts, among them CON3 VGA, CON7 SOUND, J4 UART2, J7 ESP-BUS, J8 TAPE IN, J9 TAPE OUT, Q2 BC847, U10 ESP-12E, U11 TDA1543, U16 LM311, U21 AMS1117-3.3, U7 TXB0104PW

Commit message: New schematics / revF
Parts:
- removed D10: 1N4148W, Diode_SMD:D_SOD-123, symbol Diode:1N4148W
- removed J4: UART2, Connector_PinHeader_2.54mm:PinHeader_1x05_P2.54mm_Vertical, symbol Connector_Generic:Conn_01x05
- removed J7: ESP-BUS, Connector_PinHeader_2.54mm:PinHeader_2x05_P2.54mm_Vertical, symbol Connector_Generic:Conn_02x05_Odd_Even
- removed JP3: BEEPER ON, Connector_PinHeader_2.54mm:PinHeader_1x02_P2.54mm_Vertical, symbol Jumper:Jumper_2_Open
- removed LS1: BEEPER, Buzzer_Beeper:Buzzer_12x9.5RM7.6, symbol Device:Buzzer
- removed Q2: BC847, Package_TO_SOT_SMD:SOT-23, symbol Transistor_BJT:BC847
- removed R48: 15k*, Resistor_SMD:R_0805_2012Metric_Pad1.20x1.40mm_HandSolder, symbol Device:R
- removed U7: TXB0104PW, Package_SO:TSSOP-14_4.4x5mm_P0.65mm, symbol Logic_LevelTranslator:TXB0104PW
- added J5: USB C, Connector_USB:USB_C_Receptacle_XKB_U262-16XN-4BVC11, symbol Connector:USB_C_Receptacle
- added R46, R58: 5k1, Resistor_SMD:R_0805_2012Metric_Pad1.20x1.40mm_HandSolder, symbol Device:R
- added R47, R57: 27, Resistor_SMD:R_0805_2012Metric_Pad1.20x1.40mm_HandSolder, symbol Device:R
- added R49: 10k, Resistor_SMD:R_0805_2012Metric_Pad1.15x1.40mm_HandSolder, symbol Device:R
Connections:
- net SND_BS is gone; now on net LSND_BS: U11.1 (BCK)
- net SND_DAT is gone; now on net LSND_DAT: U11.3 (DATA)
- net SND_WS is gone; now on net LSND_WS: U11.2 (WS)
- net GND: now also J5.A1 (GND), J5.A12 (GND), J5.B1 (GND), J5.B12 (GND), J5.S1 (SHIELD), R46.2, R49.1, R58.2
- net ESP_ADC: no longer names the net of U10.2 (ADC)
- net ESP_ADC: now also R49.2
- net ESP_GPIO0: no longer names the net of U10.18 (GPIO0)
- net ESP_GPIO12: no longer names the net of U10.6 (GPIO12)
- net ESP_GPIO14: no longer names the net of U10.5 (GPIO14)
- net ESP_GPIO16: no longer names the net of U10.4 (GPIO16)
- net ESP_GPIO2: no longer names the net of U10.17 (GPIO2)
- net ESP_GPIO4: no longer names the net of U10.19 (GPIO4)
- net ESP_GPIO5: no longer names the net of U10.20 (GPIO5)
- new net: J5.B5 (CC2), R46.1
- new net: J5.A5 (CC1), R58.1
- new net D+: J5.A6 (D+), J5.B6 (D+), R57.1
- new net D-: J5.A7 (D-), J5.B7 (D-), R47.1
- new net USB_D+: R57.2
- new net USB_D-: R47.2
- new net VBUS: J5.A4 (VBUS), J5.A9 (VBUS), J5.B4 (VBUS), J5.B9 (VBUS)
- no-connect marks 14 -> 31

Commit message: revF wip
Parts:
- removed C58: 100n, Capacitor_SMD:C_0805_2012Metric_Pad1.18x1.45mm_HandSolder, symbol Device:C
- R62: renamed from R49; footprint Resistor_SMD:R_0805_2012Metric_Pad1.15x1.40mm_HandSolder -> Resistor_SMD:R_0805_2012Metric_Pad1.20x1.40mm_HandSolder
- renumbered C55 to C70, C56 to C71, C54 to C72, C57 to C73, C13 to C74, C63 to C76, C1 to C77, C2 to C78, CON3 to CON8, J8 to J5, J9 to J6, J5 to J7, R30 to R61, R31 to R63, R62 to R64, R80 to R65, R81 to R66, R82 to R67, R83 to R68, R32 to R69, R84 to R70, R25 to R71, R26 to R72, R27 to R73, R46 to R74, R47 to R75, R57 to R76, R58 to R77, R10 to R78, R11 to R79, R12 to R80, R13 to R81, R14 to R82, R15 to R83, R16 to R84, R17 to R85, R18 to R86, R53 to R87, R19 to R88, R20 to R89, U10 to U18, U21 to U19, U16 to U20, U11 to U21

Commit message: revF routed
Parts:
- removed C77, C78: 10uF, Capacitor_SMD:C_0805_2012Metric_Pad1.15x1.40mm_HandSolder, symbol Device:C
- removed U21: TDA1543, Package_DIP:DIP-8_W7.62mm, symbol tda1543:TDA1543
- added C25, C48, C52: 100n, Capacitor_SMD:C_0805_2012Metric_Pad1.18x1.45mm_HandSolder, symbol Device:C
- added C26: 10uF, Capacitor_SMD:C_0805_2012Metric_Pad1.18x1.45mm_HandSolder, symbol Device:C
- added C29, C31: 47uF, Capacitor_SMD:CP_Elec_5x5.9, symbol Device:C_Polarized_Small
- added R90: 100, Resistor_SMD:R_0805_2012Metric_Pad1.20x1.40mm_HandSolder, symbol Device:R
- added U21: UDA1334ATS, Package_SO:SSOP-16_4.4x5.2mm_P0.65mm, symbol Audio:UDA1334ATS
- R71: value 820 -> 220k; footprint Resistor_SMD:R_0805_2012Metric_Pad1.15x1.40mm_HandSolder -> Resistor_SMD:R_0805_2012Metric_Pad1.20x1.40mm_HandSolder
- R72: value 750 -> 220k; footprint Resistor_SMD:R_0805_2012Metric_Pad1.15x1.40mm_HandSolder -> Resistor_SMD:R_0805_2012Metric_Pad1.20x1.40mm_HandSolder
- R73: value 750 -> 100; footprint Resistor_SMD:R_0805_2012Metric_Pad1.15x1.40mm_HandSolder -> Resistor_SMD:R_0805_2012Metric_Pad1.20x1.40mm_HandSolder
Connections:
- net GND: now also R71.1, R72.1, C25.2, C26.2, C48.2, C52.2, U21.10 (PLL0), U21.11 (SFOR0), U21.15 (VSSA), U21.5 (VSSD), U21.6 (SYSCLK/PLL1), U21.7 (SFOR1), U21.8 (MUTE), U21.9 (DEEM/CLKOUT); no longer R71.2, R72.2, R73.2
- net LSND_BS: now also U21.1 (BCK)
- net LSND_DAT: now also U21.3 (DATAI)
- net LSND_WS: now also U21.2 (WS)
- net SND_L: now also C52.1, R90.2
- net SND_R: now also R73.2, C48.1
- net VCC3_3: now also U21.13 (VDDA), U21.4 (VDDD)
- net at R73.1: now also R71.2, C29.2
- new net: C25.1, C26.1, U21.12 (Vref(DAC))
- new net: C31.1, U21.16 (VOUTR)
- new net: C31.2, R72.2, R90.1
- new net: C29.1, U21.14 (VOUTL)
Other:
- moved on the sheet: CON7, CON8, R78, R79, R80, R81, R82, R83, R84, R85, R86, R87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

Commit message: Updated revF hw and docs
Parts:
- added JP3: VBUS, Connector_PinHeader_2.54mm:PinHeader_1x02_P2.54mm_Vertical, symbol Jumper:Jumper_2_Open
Connections:
- net VBUS: now also JP3.1 (A)
- net VCC: now also JP3.2 (B)
Changed lines of the file:
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@@
 	(wire
 		(pts
+			(xy 135.89 180.34) (xy 138.43 180.34)
+		)
+		(stroke
+			(width 0)
+			(type default)
+		)
+	)
+	(wire
+		(pts
 			(xy 214.63 114.3) (xy 213.36 114.3)
 		)
@@
 	(wire
 		(pts
+			(xy 148.59 180.34) (xy 151.13 180.34)
+		)
+		(stroke
+			(width 0)
+			(type default)
+		)
+	)
+	(wire
+		(pts
 			(xy 236.22 111.76) (xy 227.33 111.76)
 		)
@@
 		)
 	)
+	(global_label "VBUS"
+		(shape input)
+		(at 135.89 180.34 180)
+		(fields_autoplaced yes)
+		(effects
+			(font
+				(size 1.27 1.27)
+			)
+			(justify right)
+		)
+		(property "Intersheetrefs" "${INTERSHEET_REFS}"
+			(at 128.6604 180.34 0)
+			(effects
+				(font
+					(size 1.27 1.27)
+				)
+				(justify right)
+				(hide yes)
+			)
+		)
+	)
 	(global_label "SND_R"
 		(shape input)
@@
 	)
 	(symbol
+		(lib_id "Jumper:Jumper_2_Open")
+		(at 143.51 180.34 0)
+		(unit 1)
+		(exclude_from_sim no)
+		(in_bom yes)
+		(on_board yes)
+		(dnp no)
+		(fields_autoplaced yes)
+		(property "Reference" "JP3"
+			(at 143.51 173.99 0)
+			(effects
+				(font
+					(size 1.27 1.27)
+				)
+			)
+		)
+		(property "Value" "VBUS"
+			(at 143.51 176.53 0)
+			(effects
+				(font
+					(size 1.27 1.27)
+				)
+			)
+		)
+		(property "Footprint" "Connector_PinHeader_2.54mm:PinHeader_1x02_P2.54mm_Vertical"
+			(at 143.51 180.34 0)
+			(effects
+				(font
+					(size 1.27 1.27)
+				)
+				(hide yes)
+			)
+		)
+		(property "Datasheet" "~"
+			(at 143.51 180.34 0)
+			(effects
+				(font
+					(size 1.27 1.27)
+				)
+				(hide yes)
+			)
+		)
+		(property "Description" ""
+			(at 143.51 180.34 0)
+			(effects
+				(font
+					(size 1.27 1.27)
+				)
+			)
+		)
+		(pin "1"
+		)
+		(pin "2"
+		)
+		(instances
+			(project "karabas-pro-revF"
+				(path "/0fa36eda-2d7d-4199-a7a1-2cda6b0cd120/7f4e7edd-196d-4c95-a36b-79063a0e6ab2"
+					(reference "JP3")
+					(unit 1)
+				)
+			)
+		)
+	)
+	(symbol
 		(lib_id "Device:R")
 		(at 163.83 115.57 90)
@@
 	)
 	(symbol
+		(lib_id "power:VCC")
+		(at 151.13 180.34 270)
+		(unit 1)
+		(exclude_from_sim no)
+		(in_bom yes)
+		(on_board yes)
+		(dnp no)
+		(property "Reference" "#PWR034"
+			(at 147.32 180.34 0)
+			(effects
+				(font
+					(size 1.27 1.27)
+				)
+				(hide yes)
+			)
+		)
+		(property "Value" "VCC"
+			(at 156.972 180.34 90)
+			(effects
+				(font
+					(size 1.27 1.27)
+				)
+			)
+		)
+		(property "Footprint" ""
+			(at 151.13 180.34 0)
+			(effects
+				(font
+					(size 1.27 1.27)
+				)
+				(hide yes)
+			)
+		)
+		(property "Datasheet" ""
+			(at 151.13 180.34 0)
+			(effects
+				(font
+					(size 1.27 1.27)
+				)
+				(hide yes)
+			)
+		)
+		(property "Description" ""
+			(at 151.13 180.34 0)
+			(effects
+				(font
+					(size 1.27 1.27)
+				)
+			)
+		)
+		(pin "1"
+		)
+		(instances
+			(project "karabas-pro-revF"
+				(path "/0fa36eda-2d7d-4199-a7a1-2cda6b0cd120/7f4e7edd-196d-4c95-a36b-79063a0e6ab2"
+					(reference "#PWR034")
+					(unit 1)
+				)
+			)
+		)
+	)
+	(symbol
 		(lib_id "Device:R")
 		(at 40.64 43.18 180)
@@
 			)
 		)
-		(property "Datasheet" " ~"
+		(property "Datasheet" "~"
 			(at 219.71 106.68 0)
 			(effects

Commit message: Updated revF
Parts:
- C26: value 10uF -> 10u
- C29, C31: value 47uF -> 47u
- C72: value 100uF -> 100u
- CON8: footprint Connector_Dsub:DSUB-15-HD_Female_Horizontal_P2.29x1.98mm_EdgePinOffset3.03mm_Housed_MountingHolesOffset4.94mm -> Connector_Dsub:DSUB-15-HD_Socket_Horizontal_P2.29x1.90mm_EdgePinOffset3.03mm_Housed_MountingHolesOffset4.94mm
- R61, R63, R78, R79, R80, R81, R82, R83, R84, R85, R86, R87: footprint Resistor_SMD:R_0805_2012Metric_Pad1.15x1.40mm_HandSolder -> Resistor_SMD:R_0805_2012Metric_Pad1.20x1.40mm_HandSolder
- R69: value 33 -> 27; footprint Resistor_SMD:R_0805_2012Metric_Pad1.15x1.40mm_HandSolder -> Resistor_SMD:R_0805_2012Metric_Pad1.20x1.40mm_HandSolder
- R88, R89: value 75 -> 100; footprint Resistor_SMD:R_0805_2012Metric_Pad1.15x1.40mm_HandSolder -> Resistor_SMD:R_0805_2012Metric_Pad1.20x1.40mm_HandSolder
Changed lines of the file:
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@@
 			)
 		)
-		(property "Footprint" "Resistor_SMD:R_0805_2012Metric_Pad1.15x1.40mm_HandSolder"
+		(property "Footprint" "Resistor_SMD:R_0805_2012Metric_Pad1.20x1.40mm_HandSolder"
 			(at 33.528 43.18 90)
 			(effects
@@
 			)
 		)
-		(property "Footprint" "Resistor_SMD:R_0805_2012Metric_Pad1.15x1.40mm_HandSolder"
+		(property "Footprint" "Resistor_SMD:R_0805_2012Metric_Pad1.20x1.40mm_HandSolder"
 			(at 218.44 131.318 90)
 			(effects
@@
 			)
 		)
-		(property "Value" "47uF"
+		(property "Value" "47u"
 			(at 162.306 50.8 90)
 			(effects
@@
 			)
 		)
-		(property "Footprint" "Resistor_SMD:R_0805_2012Metric_Pad1.15x1.40mm_HandSolder"
+		(property "Footprint" "Resistor_SMD:R_0805_2012Metric_Pad1.20x1.40mm_HandSolder"
 			(at 218.44 116.078 90)
 			(effects
@@
 			)
 		)
-		(property "Value" "100uF"
+		(property "Value" "100u"
 			(at 56.3372 35.306 0)
 			(effects
@@
 			)
 		)
-		(property "Footprint" "Resistor_SMD:R_0805_2012Metric_Pad1.15x1.40mm_HandSolder"
+		(property "Footprint" "Resistor_SMD:R_0805_2012Metric_Pad1.20x1.40mm_HandSolder"
 			(at 42.418 43.18 90)
 			(effects
@@
 			)
 		)
-		(property "Footprint" "Resistor_SMD:R_0805_2012Metric_Pad1.15x1.40mm_HandSolder"
+		(property "Footprint" "Resistor_SMD:R_0805_2012Metric_Pad1.20x1.40mm_HandSolder"
 			(at 218.44 108.458 90)
 			(effects
@@
 			)
 		)
-		(property "Footprint" "Resistor_SMD:R_0805_2012Metric_Pad1.15x1.40mm_HandSolder"
+		(property "Footprint" "Resistor_SMD:R_0805_2012Metric_Pad1.20x1.40mm_HandSolder"
 			(at 218.44 145.288 90)
 			(effects
@@
 			)
 		)
-		(property "Footprint" "Resistor_SMD:R_0805_2012Metric_Pad1.15x1.40mm_HandSolder"
+		(property "Footprint" "Resistor_SMD:R_0805_2012Metric_Pad1.20x1.40mm_HandSolder"
 			(at 218.44 138.938 90)
 			(effects
@@
 			)
 		)
-		(property "Value" "75"
+		(property "Value" "100"
 			(at 261.62 124.46 90)
 			(effects
@@
 			)
 		)
-		(property "Footprint" "Resistor_SMD:R_0805_2012Metric_Pad1.15x1.40mm_HandSolder"
+		(property "Footprint" "Resistor_SMD:R_0805_2012Metric_Pad1.20x1.40mm_HandSolder"
 			(at 261.62 123.698 90)
 			(effects
@@
 			)
 		)
-		(property "Value" "47uF"
+		(property "Value" "47u"
 			(at 162.0139 36.83 90)
 			(effects
@@
 			)
 		)
-		(property "Footprint" "Resistor_SMD:R_0805_2012Metric_Pad1.15x1.40mm_HandSolder"
+		(property "Footprint" "Resistor_SMD:R_0805_2012Metric_Pad1.20x1.40mm_HandSolder"
 			(at 218.44 119.888 90)
 			(effects
@@
 			)
 		)
-		(property "Footprint" "Resistor_SMD:R_0805_2012Metric_Pad1.15x1.40mm_HandSolder"
+		(property "Footprint" "Resistor_SMD:R_0805_2012Metric_Pad1.20x1.40mm_HandSolder"
 			(at 218.44 100.838 90)
 			(effects
@@
 			)
 		)
-		(property "Value" "10uF"
+		(property "Value" "10u"
 			(at 170.4594 59.69 90)
 			(effects
@@
 			)
 		)
-		(property "Value" "33"
+		(property "Value" "27"
 			(at 78.74 78.74 90)
 			(effects
@@
 			)
 		)
-		(property "Footprint" "Resistor_SMD:R_0805_2012Metric_Pad1.15x1.40mm_HandSolder"
+		(property "Footprint" "Resistor_SMD:R_0805_2012Metric_Pad1.20x1.40mm_HandSolder"
 			(at 77.978 78.74 90)
 			(effects
@@
 			)
 		)
-		(property "Footprint" "Resistor_SMD:R_0805_2012Metric_Pad1.15x1.40mm_HandSolder"
+		(property "Footprint" "Resistor_SMD:R_0805_2012Metric_Pad1.20x1.40mm_HandSolder"
 			(at 218.44 123.698 90)
 			(effects
@@
 			)
 		)
-		(property "Footprint" "Connector_Dsub:DSUB-15-HD_Female_Horizontal_P2.29x1.98mm_EdgePinOffset3.03mm_Housed_MountingHolesOffset4.94mm"
+		(property "Footprint" "Connector_Dsub:DSUB-15-HD_Socket_Horizontal_P2.29x1.90mm_EdgePinOffset3.03mm_Housed_MountingHolesOffset4.94mm"
 			(at 219.71 106.68 0)
 			(effects
@@
 			)
 		)
-		(property "Footprint" "Resistor_SMD:R_0805_2012Metric_Pad1.15x1.40mm_HandSolder"
+		(property "Footprint" "Resistor_SMD:R_0805_2012Metric_Pad1.20x1.40mm_HandSolder"
 			(at 218.44 104.648 90)
 			(effects
@@
 			)
 		)
-		(property "Value" "75"
+		(property "Value" "100"
 			(at 261.62 114.3 90)
 			(effects
@@
 			)
 		)
-		(property "Footprint" "Resistor_SMD:R_0805_2012Metric_Pad1.15x1.40mm_HandSolder"
+		(property "Footprint" "Resistor_SMD:R_0805_2012Metric_Pad1.20x1.40mm_HandSolder"
 			(at 261.62 118.618 90)
 			(effects
@@
 			)
 		)
-		(property "Footprint" "Resistor_SMD:R_0805_2012Metric_Pad1.15x1.40mm_HandSolder"
+		(property "Footprint" "Resistor_SMD:R_0805_2012Metric_Pad1.20x1.40mm_HandSolder"
 			(at 218.44 135.128 90)
 			(effects

Commit message: RevF pcb
Parts:
- U21: footprint Package_SO:SSOP-16_4.4x5.2mm_P0.65mm -> footprints:SSOP-16_4.4x5.2mm_P0.65mm-extended
Changed lines of the file:
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@@
 			)
 		)
-		(property "Footprint" "Package_SO:SSOP-16_4.4x5.2mm_P0.65mm"
+		(property "Footprint" "footprints:SSOP-16_4.4x5.2mm_P0.65mm-extended"
 			(at 140.97 48.26 0)
 			(effects

Commit message: Refactored revF alpha2
Parts:
- removed JP3: VBUS, Connector_PinHeader_2.54mm:PinHeader_1x02_P2.54mm_Vertical, symbol Jumper:Jumper_2_Open
- added D9: BAT54C, Package_TO_SOT_SMD:SOT-23_Handsoldering, symbol Diode:BAT54C
Connections:
- net VBUS: now also D9.1
- net VCC: now also D9.3
- no-connect marks 31 -> 32
Changed lines of the file:
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@@
 	)
 	(no_connect
+		(at 153.67 180.34)
+	)
+	(no_connect
 		(at 44.45 69.85)
 	)
@@
 	(wire
 		(pts
-			(xy 148.59 180.34) (xy 151.13 180.34)
+			(xy 146.05 185.42) (xy 148.59 185.42)
 		)
 		(stroke
@@
 	)
 	(symbol
-		(lib_id "Jumper:Jumper_2_Open")
-		(at 143.51 180.34 0)
-		(unit 1)
-		(exclude_from_sim no)
-		(in_bom yes)
-		(on_board yes)
-		(dnp no)
-		(fields_autoplaced yes)
-		(property "Reference" "JP3"
-			(at 143.51 173.99 0)
-			(effects
-				(font
-					(size 1.27 1.27)
-				)
-			)
-		)
-		(property "Value" "VBUS"
-			(at 143.51 176.53 0)
-			(effects
-				(font
-					(size 1.27 1.27)
-				)
-			)
-		)
-		(property "Footprint" "Connector_PinHeader_2.54mm:PinHeader_1x02_P2.54mm_Vertical"
-			(at 143.51 180.34 0)
-			(effects
-				(font
-					(size 1.27 1.27)
-				)
-				(hide yes)
-			)
-		)
-		(property "Datasheet" "~"
-			(at 143.51 180.34 0)
-			(effects
-				(font
-					(size 1.27 1.27)
-				)
-				(hide yes)
-			)
-		)
-		(property "Description" ""
-			(at 143.51 180.34 0)
-			(effects
-				(font
-					(size 1.27 1.27)
-				)
-			)
-		)
-		(pin "1"
-		)
-		(pin "2"
-		)
-		(instances
-			(project "karabas-pro-revF"
-				(path "/0fa36eda-2d7d-4199-a7a1-2cda6b0cd120/7f4e7edd-196d-4c95-a36b-79063a0e6ab2"
-					(reference "JP3")
-					(unit 1)
-				)
-			)
-		)
-	)
-	(symbol
 		(lib_id "Device:R")
 		(at 163.83 115.57 90)
@@
 	(symbol
 		(lib_id "power:VCC")
-		(at 151.13 180.34 270)
+		(at 148.59 185.42 270)
 		(unit 1)
 		(exclude_from_sim no)
@@
 		(dnp no)
 		(property "Reference" "#PWR034"
-			(at 147.32 180.34 0)
+			(at 144.78 185.42 0)
 			(effects
 				(font
@@
 		)
 		(property "Value" "VCC"
-			(at 156.972 180.34 90)
+			(at 154.432 185.42 90)
 			(effects
 				(font
@@
 		)
 		(property "Footprint" ""
-			(at 151.13 180.34 0)
+			(at 148.59 185.42 0)
 			(effects
 				(font
@@
 		)
 		(property "Datasheet" ""
-			(at 151.13 180.34 0)
+			(at 148.59 185.42 0)
 			(effects
 				(font
@@
 		)
 		(property "Description" ""
-			(at 151.13 180.34 0)
+			(at 148.59 185.42 0)
 			(effects
 				(font
@@
 					(unit 1)
 				)
+			)
+		)
+	)
+	(symbol
+		(lib_id "Diode:BAT54C")
+		(at 146.05 180.34 0)
+		(unit 1)
+		(exclude_from_sim no)
+		(in_bom yes)
+		(on_board yes)
+		(dnp no)
+		(property "Reference" "D9"
+			(at 146.05 174.625 0)
+			(effects
+				(font
+					(size 1.27 1.27)
+				)
+			)
+		)
+		(property "Value" "BAT54C"
+			(at 146.05 176.9364 0)
+			(effects
+				(font
+					(size 1.27 1.27)
+				)
+			)
+		)
+		(property "Footprint" "Package_TO_SOT_SMD:SOT-23_Handsoldering"
+			(at 147.955 177.165 0)
+			(effects
+				(font
+					(size 1.27 1.27)
+				)
+				(justify left)
+				(hide yes)
+			)
+		)
+		(property "Datasheet" "http://www.diodes.com/_files/datasheets/ds11005.pdf"
+			(at 144.018 180.34 0)
+			(effects
+				(font
+					(size 1.27 1.27)
+				)
+				(hide yes)
+			)
+		)
+		(property "Description" ""
+			(at 146.05 180.34 0)
+			(effects
+				(font
+					(size 1.27 1.27)
+				)
+			)
+		)
+		(pin "1"
+		)
+		(pin "2"
+		)
+		(pin "3"
+		)
+		(instances
+			(project "karabas-pro-revF"
+				(path "/0fa36eda-2d7d-4199-a7a1-2cda6b0cd120/7f4e7edd-196d-4c95-a36b-79063a0e6ab2"
+					(reference "D9")
+					(unit 1)
+				)
