File: pcb/revF/interfaces.kicad_sch (KiCad schematic)
At the start: 52 parts, among them CON7 SOUND, CON8 VGA, J5 TAPE IN, J6 TAPE OUT, J7 USB C, U18 ESP-12E, U19 AMS1117-3.3, U20 LM311, U21 UDA1334ATS

Commit message: PCB revF a4
Parts:
- removed C29, C31: 47u, Capacitor_SMD:CP_Elec_5x5.9, symbol Device:C_Polarized_Small
- removed R71, R72: 220k, Resistor_SMD:R_0805_2012Metric_Pad1.20x1.40mm_HandSolder, symbol Device:R
- removed R73, R90: 100, Resistor_SMD:R_0805_2012Metric_Pad1.20x1.40mm_HandSolder, symbol Device:R
- removed U21: UDA1334ATS, footprints:SSOP-16_4.4x5.2mm_P0.65mm-extended, symbol Audio:UDA1334ATS
- added C29, C75, C78: 10u, Capacitor_SMD:C_0805_2012Metric_Pad1.18x1.45mm_HandSolder, symbol Device:C
- added C31: 2n2, Capacitor_SMD:C_0805_2012Metric_Pad1.18x1.45mm_HandSolder, symbol Device:C
- added C77, C79: 100n, Capacitor_SMD:C_0805_2012Metric_Pad1.18x1.45mm_HandSolder, symbol Device:C
- added R4, R5: 10k, Resistor_SMD:R_0805_2012Metric_Pad1.20x1.40mm_HandSolder, symbol Device:R
- added R7: 1k, Resistor_SMD:R_0805_2012Metric_Pad1.20x1.40mm_HandSolder, symbol Device:R
- added U21: PCM5102A, Package_SO:TSSOP-20_4.4x6.5mm_P0.65mm, symbol Audio:PCM5102A
- C48: value 100n -> 2n2
- C52: value 100n -> 2u2
Connections:
- net GND: now also C48.1, C31.1, C75.1, C77.1, C78.1, C79.1, U21.10 (DEMP), U21.11 (FLT), U21.12 (SCK), U21.16 (FMT), U21.19 (DGND), U21.3 (CPGND), U21.9 (AGND); no longer C26.2, C48.2, C52.2
- net LSND_BS: now also U21.13 (BCK)
- net LSND_DAT: now also U21.14 (DIN)
- net LSND_WS: now also U21.15 (LRCK)
- net SND_L: now also C26.1; no longer C52.1
- net SND_R: now also C29.1; no longer C48.1
- net VCC3_3: now also C25.1, R7.1, U21.1 (CPVDD), U21.20 (DVDD), U21.8 (AVDD)
- net ~{ESP_RESET}: now reaches R63.1, U18.1 (~{RST})
- net ~{ESP_BOOT}: now reaches U18.18 (GPIO0)
- new net: C29.2, C48.2, R5.2
- new net: R7.2, U21.17 (XSMT)
- new net: C26.2, C31.2, R4.2
- new net: C78.2, C79.2, U21.18 (LDOO)
- new net: R4.1, U21.6 (OUTL)
- new net: R5.1, U21.7 (OUTR)
- new net: C75.2, C77.2, U21.5 (VNEG)
- new net: C52.1, U21.4 (CAPM)
- new net: C52.2, U21.2 (CAPP)
- no-connect marks 32 -> 31
