File: pcb/revF/mcu.kicad_sch (KiCad schematic)
At the start: 64 parts, among them CON1 JOYSTICK, CON2 KEYBOARD, CON3 MOUSE, J2 I2C, Q1 IRLML2402, Q2 IRLML2402, Q3 IRLML2402, Q4 IRLML2402, U4 24LC08B, U5 W25Q128JVS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

Commit message: PCB revF a4
Parts:
- removed TP3: A1, TestPoint:TestPoint_Pad_D1.0mm, symbol Connector:TestPoint
- removed TP4: A2, TestPoint:TestPoint_Pad_D1.0mm, symbol Connector:TestPoint
- removed TP5: A3, TestPoint:TestPoint_Pad_D1.0mm, symbol Connector:TestPoint
- removed U6: DS3231MZ, Package_SO:SOIC-8_3.9x4.9mm_P1.27mm, symbol Timer_RTC:DS3231MZ
- added U2: DS1307Z+, Package_SO:SOIC-8_3.9x4.9mm_P1.27mm, symbol Timer_RTC:DS1307Z+
- added Y2: 32768, Crystal:Crystal_C26-LF_D2.1mm_L6.5mm_Horizontal_1EP_style2, symbol Device:Crystal_GND3_Small
Connections:
- net GND: now also U2.4 (GND), Y2.3
- net I2C_SCL: now also U2.6 (SCL)
- net I2C_SDA: now also U2.5 (SDA)
- net VBat: now also U2.3 (VBAT)
- net VCC: now also C2.1, U2.8 (VCC)
- net VCC3_3: no longer C2.1
- new net: U2.1 (X1), Y2.1
- new net: U2.2 (X2), Y2.2
- no-connect marks 9 -> 10
Other:
- moved on the sheet: BT1, C1, C2, U4
