File: pcb/revF/karabas-pro-revF.kicad_sch (KiCad schematic)
At the start: 8 parts

Commit message: New schematics / revF
Changed lines of the file:
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@@
     (fill (type none))
   )
-  (rectangle (start 104.14 90.17) (end 116.84 90.17)
+  (rectangle (start 196.85 151.13) (end 241.3 151.13)
     (stroke (width 0) (type default))
     (fill (type none))
@@
     (fill (type none))
   )
-  (rectangle (start 104.14 120.65) (end 116.84 120.65)
-    (stroke (width 0) (type default))
-    (fill (type none))
-  )
   (rectangle (start 196.85 130.81) (end 241.3 130.81)
     (stroke (width 0) (type default))
@@
     (stroke (width 0) (type default))
     (fill (type none))
-  )
-  (text_box "BUZZER"
-    (at 74.93 116.84 0) (size 29.21 7.62)
-    (stroke (width 0) (type default))
-    (fill (type none))
-    (effects (font (size 1.27 1.27)))
   )
   (text_box "PS/2 Keyboard"
@@
   )
   (text_box "ESP8266"
-    (at 74.93 86.36 0) (size 29.21 7.62)
+    (at 241.3 147.32 0) (size 29.21 7.62)
     (stroke (width 0) (type default))
     (fill (type none))
@@
     (effects (font (size 1.27 1.27)))
   )
-  (text_box "SRAM 6MB"
+  (text_box "SRAM 2MB"
     (at 74.93 55.88 0) (size 29.21 7.62)
     (stroke (width 0) (type default))
@@
     (effects (font (size 1.27 1.27)))
   )
-  (text_box "FPGA\nEP4CE10"
-    (at 116.84 45.72 0) (size 46.99 99.06)
+  (text_box "FPGA\nEP4CE22"
+    (at 116.84 45.72 0) (size 46.99 109.22)
     (stroke (width 0) (type default))
     (fill (type none))
@@
     (effects (font (size 1.27 1.27)))
   )
-  (text_box "AVR\nATMEGA328"
-    (at 179.07 66.04 0) (size 17.78 78.74)
+  (text_box "MCU\nRP2040"
+    (at 179.07 66.04 0) (size 17.78 88.9)
     (stroke (width 0) (type default))
     (fill (type none))
@@
     (effects (font (size 1.27 1.27) (thickness 0.254) bold) (justify left bottom))
   )
-  (text "UART" (at 107.95 90.17 0)
+  (text "UART" (at 215.9 151.13 0)
     (effects (font (size 1.27 1.27)) (justify left bottom))
   )

Commit message: revF wip
Parts:
- added LOGO_ANDY1: Logo_Open_Hardware_Small, footprints:andy_karpov_logo4_silk, symbol Graphic:Logo_Open_Hardware_Small
- added LOGO_BOTTOM1: Logo_Open_Hardware_Small, footprints:karabas_pro_logo4_copper, symbol Graphic:Logo_Open_Hardware_Small
- added LOGO_TOP1: Logo_Open_Hardware_Small, footprints:karabas_pro_logo2-coppermask, symbol Graphic:Logo_Open_Hardware_Small
- renumbered H5 to H2, H2 to H3, H6 to H4, H3 to H5, H7 to H6, H4 to H7

Commit message: revF routed
Parts:
- LOGO_TOP1: footprint footprints:karabas_pro_logo2-coppermask -> footprints:karabas_pro_logo4_copper
Other:
- note added: "CONF"

Commit message: Updated revF hw and docs
Parts:
- H1, H2, H3, H4, H5, H6, H7, H8: now left out of the parts list
Other:
- note added: "I2C"
Changed lines of the file:
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@@
+		)
+	)
+	(text "I2C"
+		(exclude_from_sim no)
+		(at 215.9 89.662 0)
+		(effects
+			(font
+				(size 1.27 1.27)
+			)
+			(justify left bottom)
 		)
 	)
@@
 		)
 	)
-	(text_box "RTC"
+	(text_box "RTC, EEPROM"
 		(exclude_from_sim no)
 		(at 241.3 86.36 0)
@@
 		(stroke
 			(width 0)
-			(type default)
+			(type solid)
 		)
 		(fill
@@
 		(unit 1)
 		(exclude_from_sim no)
-		(in_bom yes)
+		(in_bom no)
 		(on_board yes)
 		(dnp no)
@@
 		(unit 1)
 		(exclude_from_sim no)
-		(in_bom yes)
+		(in_bom no)
 		(on_board yes)
 		(dnp no)
@@
 		(unit 1)
 		(exclude_from_sim no)
-		(in_bom yes)
+		(in_bom no)
 		(on_board yes)
 		(dnp no)
@@
 		(unit 1)
 		(exclude_from_sim no)
-		(in_bom yes)
+		(in_bom no)
 		(on_board yes)
 		(dnp no)
@@
 		(unit 1)
 		(exclude_from_sim no)
-		(in_bom yes)
+		(in_bom no)
 		(on_board yes)
 		(dnp no)
@@
 		(unit 1)
 		(exclude_from_sim no)
-		(in_bom yes)
+		(in_bom no)
 		(on_board yes)
 		(dnp no)
@@
 		(unit 1)
 		(exclude_from_sim no)
-		(in_bom yes)
+		(in_bom no)
 		(on_board yes)
 		(dnp no)
@@
 		(unit 1)
 		(exclude_from_sim no)
-		(in_bom yes)
+		(in_bom no)
 		(on_board yes)
 		(dnp no)

Commit message: PCB RevF a3
Other:
- note added: "Karabas Pro Rev.${REVISION} simplified block diagram"
- note removed: "Karabas Pro simplified block diagram"
Changed lines of the file:
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@@
 	(title_block
 		(title "Karabas Pro")
-		(date "2024-05-01")
-		(rev "F")
+		(date "2025-10-10")
+		(rev "F a3")
 	)
 	(rectangle
@@
 		)
 	)
-	(text "Karabas Pro simplified block diagram"
+	(text "Karabas Pro Rev.${REVISION} simplified block diagram"
 		(exclude_from_sim no)
 		(at 74.93 40.64 0)

Commit message: PCB revF a4
Changed lines of the file:
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@@
 	(title_block
 		(title "Karabas Pro")
-		(date "2025-10-10")
-		(rev "F a3")
+		(date "2026-02-23")
+		(rev "F a4")
 	)
 	(rectangle
