File: pcb/revF/memory.kicad_sch (KiCad schematic)
At the start: 3 parts, among them U19 CY62167EV30LL, U2 CY62167EV30LL, U20 BS62LV1600

Commit message: New schematics / revF
Parts:
- removed U19: CY62167EV30LL, Package_SO:TSOP-I-48_18.4x12mm_P0.5mm, symbol retro:CY62167ELL
- removed U20: BS62LV1600, Package_SO:TSOP-II-44_10.16x18.41mm_P0.8mm, symbol retro:BS62LV1600
Connections:
- net ~{MRD} is gone; now on net GND: U2.28 (~{OE})
- net ~{RAMCE1} is gone; now on net GND: U2.26 (~{CE1})
- no-connect marks 18 -> 9

Commit message: revF wip
Parts:
- renumbered U2 to U3
Changed lines of the file:
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@@
   (symbol (lib_id "retro:CY62167ELL") (at 66.04 73.66 0) (unit 1)
     (in_bom yes) (on_board yes) (dnp no)
-    (property "Reference" "U2" (at 66.04 35.1282 0)
+    (property "Reference" "U3" (at 66.04 35.1282 0)
       (effects (font (size 1.27 1.27)))
     )
@@
       (project "karabas-pro-revF"
         (path "/0fa36eda-2d7d-4199-a7a1-2cda6b0cd120/cdc55636-5730-4b5f-b94c-1678f6b9ec0f"
-          (reference "U2") (unit 1)
+          (reference "U3") (unit 1)
         )
       )
@@
   (symbol (lib_id "vcc33:VCC3_3") (at 49.53 110.49 90) (mirror x) (unit 1)
     (in_bom yes) (on_board yes) (dnp no)
-    (property "Reference" "#PWR0149" (at 53.34 110.49 0)
+    (property "Reference" "#PWR026" (at 53.34 110.49 0)
       (effects (font (size 1.27 1.27)) hide)
     )
@@
       (project "karabas-pro-revF"
         (path "/0fa36eda-2d7d-4199-a7a1-2cda6b0cd120/cdc55636-5730-4b5f-b94c-1678f6b9ec0f"
-          (reference "#PWR0149") (unit 1)
+          (reference "#PWR026") (unit 1)
         )
       )
@@
   (symbol (lib_id "vcc33:VCC3_3") (at 82.55 105.41 270) (unit 1)
     (in_bom yes) (on_board yes) (dnp no)
-    (property "Reference" "#PWR0148" (at 78.74 105.41 0)
+    (property "Reference" "#PWR027" (at 78.74 105.41 0)
       (effects (font (size 1.27 1.27)) hide)
     )
@@
       (project "karabas-pro-revF"
         (path "/0fa36eda-2d7d-4199-a7a1-2cda6b0cd120/cdc55636-5730-4b5f-b94c-1678f6b9ec0f"
-          (reference "#PWR0148") (unit 1)
+          (reference "#PWR027") (unit 1)
         )
       )
@@
   (symbol (lib_id "power:GND") (at 82.55 110.49 90) (unit 1)
     (in_bom yes) (on_board yes) (dnp no)
-    (property "Reference" "#PWR0153" (at 88.9 110.49 0)
+    (property "Reference" "#PWR028" (at 88.9 110.49 0)
       (effects (font (size 1.27 1.27)) hide)
     )
@@
       (project "karabas-pro-revF"
         (path "/0fa36eda-2d7d-4199-a7a1-2cda6b0cd120/cdc55636-5730-4b5f-b94c-1678f6b9ec0f"
-          (reference "#PWR0153") (unit 1)
+          (reference "#PWR028") (unit 1)
         )
       )
@@
   (symbol (lib_id "power:GND") (at 49.53 95.25 270) (mirror x) (unit 1)
     (in_bom yes) (on_board yes) (dnp no)
-    (property "Reference" "#PWR0155" (at 43.18 95.25 0)
+    (property "Reference" "#PWR024" (at 43.18 95.25 0)
       (effects (font (size 1.27 1.27)) hide)
     )
@@
       (project "karabas-pro-revF"
         (path "/0fa36eda-2d7d-4199-a7a1-2cda6b0cd120/cdc55636-5730-4b5f-b94c-1678f6b9ec0f"
-          (reference "#PWR0155") (unit 1)
+          (reference "#PWR024") (unit 1)
         )
       )
@@
   (symbol (lib_id "power:GND") (at 49.53 107.95 270) (mirror x) (unit 1)
     (in_bom yes) (on_board yes) (dnp no)
-    (property "Reference" "#PWR022" (at 43.18 107.95 0)
+    (property "Reference" "#PWR025" (at 43.18 107.95 0)
       (effects (font (size 1.27 1.27)) hide)
     )
@@
       (project "karabas-pro-revF"
         (path "/0fa36eda-2d7d-4199-a7a1-2cda6b0cd120/cdc55636-5730-4b5f-b94c-1678f6b9ec0f"
-          (reference "#PWR022") (unit 1)
+          (reference "#PWR025") (unit 1)
         )
       )
