File: pcb/revF/peripherial.kicad_sch (KiCad schematic)
At the start: 5 parts, among them U4 EPM3128ATC100-10N

Commit message: revF wip
Parts:
- renumbered R38 to R29, R39 to R30, R78 to R31, R79 to R32, U4 to U10
Changed lines of the file:
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@@
   (symbol (lib_id "Device:R") (at 53.34 49.53 180) (unit 1)
     (in_bom yes) (on_board yes) (dnp no)
-    (property "Reference" "R39" (at 53.34 49.53 90)
+    (property "Reference" "R30" (at 53.34 49.53 90)
       (effects (font (size 1.27 1.27)))
     )
@@
       (project "karabas-pro-revF"
         (path "/0fa36eda-2d7d-4199-a7a1-2cda6b0cd120/9d189882-b488-48d5-809b-5b9cce0183ab"
-          (reference "R39") (unit 1)
+          (reference "R30") (unit 1)
         )
       )
@@
   (symbol (lib_id "Device:R") (at 100.33 39.37 180) (unit 1)
     (in_bom yes) (on_board yes) (dnp no)
-    (property "Reference" "R79" (at 100.33 39.37 90)
+    (property "Reference" "R32" (at 100.33 39.37 90)
       (effects (font (size 1.27 1.27)))
     )
@@
       (project "karabas-pro-revF"
         (path "/0fa36eda-2d7d-4199-a7a1-2cda6b0cd120/9d189882-b488-48d5-809b-5b9cce0183ab"
-          (reference "R79") (unit 1)
+          (reference "R32") (unit 1)
         )
       )
@@
   (symbol (lib_id "retro:EPM7128STC100") (at 100.33 90.17 0) (unit 1)
     (in_bom yes) (on_board yes) (dnp no)
-    (property "Reference" "U4" (at 99.06 86.36 0)
+    (property "Reference" "U10" (at 99.06 86.36 0)
       (effects (font (size 1.27 1.27)) (justify left))
     )
@@
       (project "karabas-pro-revF"
         (path "/0fa36eda-2d7d-4199-a7a1-2cda6b0cd120/9d189882-b488-48d5-809b-5b9cce0183ab"
-          (reference "U4") (unit 1)
+          (reference "U10") (unit 1)
         )
       )
@@
   (symbol (lib_id "vcc33:VCC3_3") (at 46.99 45.72 0) (unit 1)
     (in_bom yes) (on_board yes) (dnp no)
-    (property "Reference" "#PWR081" (at 46.99 49.53 0)
+    (property "Reference" "#PWR079" (at 46.99 49.53 0)
       (effects (font (size 1.27 1.27)) hide)
     )
@@
       (project "karabas-pro-revF"
         (path "/0fa36eda-2d7d-4199-a7a1-2cda6b0cd120/9d189882-b488-48d5-809b-5b9cce0183ab"
-          (reference "#PWR081") (unit 1)
+          (reference "#PWR079") (unit 1)
         )
       )
@@
   (symbol (lib_id "Device:R") (at 92.71 39.37 180) (unit 1)
     (in_bom yes) (on_board yes) (dnp no)
-    (property "Reference" "R78" (at 92.71 39.37 90)
+    (property "Reference" "R31" (at 92.71 39.37 90)
       (effects (font (size 1.27 1.27)))
     )
@@
       (project "karabas-pro-revF"
         (path "/0fa36eda-2d7d-4199-a7a1-2cda6b0cd120/9d189882-b488-48d5-809b-5b9cce0183ab"
-          (reference "R78") (unit 1)
+          (reference "R31") (unit 1)
         )
       )
@@
   (symbol (lib_id "Device:R") (at 46.99 49.53 180) (unit 1)
     (in_bom yes) (on_board yes) (dnp no)
-    (property "Reference" "R38" (at 46.99 49.53 90)
+    (property "Reference" "R29" (at 46.99 49.53 90)
       (effects (font (size 1.27 1.27)))
     )
@@
       (project "karabas-pro-revF"
         (path "/0fa36eda-2d7d-4199-a7a1-2cda6b0cd120/9d189882-b488-48d5-809b-5b9cce0183ab"
-          (reference "R38") (unit 1)
+          (reference "R29") (unit 1)
         )
       )
@@
   (symbol (lib_id "power:GND") (at 53.34 45.72 180) (unit 1)
     (in_bom yes) (on_board yes) (dnp no)
-    (property "Reference" "#PWR082" (at 53.34 39.37 0)
+    (property "Reference" "#PWR080" (at 53.34 39.37 0)
       (effects (font (size 1.27 1.27)) hide)
     )
@@
       (project "karabas-pro-revF"
         (path "/0fa36eda-2d7d-4199-a7a1-2cda6b0cd120/9d189882-b488-48d5-809b-5b9cce0183ab"
-          (reference "#PWR082") (unit 1)
-        )
-      )
+          (reference "#PWR080") (unit 1)
+        )
+      )

Commit message: Updated revF
Parts:
- R29, R30, R31, R32: footprint Resistor_SMD:R_0805_2012Metric_Pad1.15x1.40mm_HandSolder -> Resistor_SMD:R_0805_2012Metric_Pad1.20x1.40mm_HandSolder
Changed lines of the file:
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@@
 			)
 		)
-		(property "Footprint" "Resistor_SMD:R_0805_2012Metric_Pad1.15x1.40mm_HandSolder"
+		(property "Footprint" "Resistor_SMD:R_0805_2012Metric_Pad1.20x1.40mm_HandSolder"
 			(at 55.118 49.53 90)
 			(effects
@@
 			)
 		)
-		(property "Footprint" "Resistor_SMD:R_0805_2012Metric_Pad1.15x1.40mm_HandSolder"
+		(property "Footprint" "Resistor_SMD:R_0805_2012Metric_Pad1.20x1.40mm_HandSolder"
 			(at 102.108 39.37 90)
 			(effects
@@
 			)
 		)
-		(property "Footprint" "Resistor_SMD:R_0805_2012Metric_Pad1.15x1.40mm_HandSolder"
+		(property "Footprint" "Resistor_SMD:R_0805_2012Metric_Pad1.20x1.40mm_HandSolder"
 			(at 94.488 39.37 90)
 			(effects
@@
 			)
 		)
-		(property "Footprint" "Resistor_SMD:R_0805_2012Metric_Pad1.15x1.40mm_HandSolder"
+		(property "Footprint" "Resistor_SMD:R_0805_2012Metric_Pad1.20x1.40mm_HandSolder"
 			(at 48.768 49.53 90)
 			(effects
