File: pcb/revF/storage.kicad_sch (KiCad schematic)
At the start: 18 parts, among them CON1 CF CARD, CON2 SD CARD, CON9 uSD CARD, Q1 BC856

Commit message: New schematics / revF
Parts:
- removed CON9: uSD CARD, footprints:Conn_uSDcard, symbol retro:MicroSD_Molex
Connections:
- net ~{SD_DET}: no longer names the net of CON2.10 (CARD_DETECT), R52.1
Other:
- moved on the sheet: CON2, R36, R37, R52

Commit message: revF wip
Parts:
- renumbered CON2 to CON5, CON1 to CON6, D4 to D6, D6 to D7, Q1 to Q5, R36 to R34, R37 to R35, R54 to R36, R55 to R37, R52 to R38, R74 to R39, R75 to R40, R70 to R41, R71 to R42, R72 to R43, R73 to R44, R76 to R45

Commit message: Updated revF hw and docs
Parts:
- R36, R37: value 470 -> 1k
Changed lines of the file:
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@@
 			)
 		)
-		(property "Value" "470"
+		(property "Value" "1k"
 			(at 60.96 153.67 90)
 			(effects
@@
 			)
 		)
-		(property "Value" "470"
+		(property "Value" "1k"
 			(at 60.96 176.53 90)
 			(effects

Commit message: Updated revF
Parts:
- Q5: footprint Package_TO_SOT_SMD:SOT-23 -> Package_TO_SOT_SMD:SOT-23_Handsoldering
- R34, R35, R36, R37, R38, R39, R40, R41, R42, R43, R44, R45: footprint Resistor_SMD:R_0805_2012Metric_Pad1.15x1.40mm_HandSolder -> Resistor_SMD:R_0805_2012Metric_Pad1.20x1.40mm_HandSolder
Changed lines of the file:
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@@
 			)
 		)
-		(property "Footprint" "Resistor_SMD:R_0805_2012Metric_Pad1.15x1.40mm_HandSolder"
+		(property "Footprint" "Resistor_SMD:R_0805_2012Metric_Pad1.20x1.40mm_HandSolder"
 			(at 218.44 138.938 90)
 			(effects
@@
 			)
 		)
-		(property "Footprint" "Resistor_SMD:R_0805_2012Metric_Pad1.15x1.40mm_HandSolder"
+		(property "Footprint" "Resistor_SMD:R_0805_2012Metric_Pad1.20x1.40mm_HandSolder"
 			(at 196.85 94.488 90)
 			(effects
@@
 			)
 		)
-		(property "Footprint" "Resistor_SMD:R_0805_2012Metric_Pad1.15x1.40mm_HandSolder"
+		(property "Footprint" "Resistor_SMD:R_0805_2012Metric_Pad1.20x1.40mm_HandSolder"
 			(at 100.838 41.91 90)
 			(effects
@@
 			)
 		)
-		(property "Footprint" "Resistor_SMD:R_0805_2012Metric_Pad1.15x1.40mm_HandSolder"
+		(property "Footprint" "Resistor_SMD:R_0805_2012Metric_Pad1.20x1.40mm_HandSolder"
 			(at 41.91 67.818 90)
 			(effects
@@
 			)
 		)
-		(property "Footprint" "Resistor_SMD:R_0805_2012Metric_Pad1.15x1.40mm_HandSolder"
+		(property "Footprint" "Resistor_SMD:R_0805_2012Metric_Pad1.20x1.40mm_HandSolder"
 			(at 60.96 152.908 90)
 			(effects
@@
 			)
 		)
-		(property "Footprint" "Resistor_SMD:R_0805_2012Metric_Pad1.15x1.40mm_HandSolder"
+		(property "Footprint" "Resistor_SMD:R_0805_2012Metric_Pad1.20x1.40mm_HandSolder"
 			(at 218.44 132.588 90)
 			(effects
@@
 			)
 		)
-		(property "Footprint" "Resistor_SMD:R_0805_2012Metric_Pad1.15x1.40mm_HandSolder"
+		(property "Footprint" "Resistor_SMD:R_0805_2012Metric_Pad1.20x1.40mm_HandSolder"
 			(at 196.85 98.298 90)
 			(effects
@@
 			)
 		)
-		(property "Footprint" "Package_TO_SOT_SMD:SOT-23"
+		(property "Footprint" "Package_TO_SOT_SMD:SOT-23_Handsoldering"
 			(at 57.15 154.305 0)
 			(effects
@@
 			)
 		)
-		(property "Footprint" "Resistor_SMD:R_0805_2012Metric_Pad1.15x1.40mm_HandSolder"
+		(property "Footprint" "Resistor_SMD:R_0805_2012Metric_Pad1.20x1.40mm_HandSolder"
 			(at 43.688 41.91 90)
 			(effects
@@
 			)
 		)
-		(property "Footprint" "Resistor_SMD:R_0805_2012Metric_Pad1.15x1.40mm_HandSolder"
+		(property "Footprint" "Resistor_SMD:R_0805_2012Metric_Pad1.20x1.40mm_HandSolder"
 			(at 218.44 151.638 90)
 			(effects
@@
 			)
 		)
-		(property "Footprint" "Resistor_SMD:R_0805_2012Metric_Pad1.15x1.40mm_HandSolder"
+		(property "Footprint" "Resistor_SMD:R_0805_2012Metric_Pad1.20x1.40mm_HandSolder"
 			(at 60.96 175.768 90)
 			(effects
@@
 			)
 		)
-		(property "Footprint" "Resistor_SMD:R_0805_2012Metric_Pad1.15x1.40mm_HandSolder"
+		(property "Footprint" "Resistor_SMD:R_0805_2012Metric_Pad1.20x1.40mm_HandSolder"
 			(at 241.3 86.868 90)
 			(effects
@@
 			)
 		)
-		(property "Footprint" "Resistor_SMD:R_0805_2012Metric_Pad1.15x1.40mm_HandSolder"
+		(property "Footprint" "Resistor_SMD:R_0805_2012Metric_Pad1.20x1.40mm_HandSolder"
 			(at 218.44 145.288 90)
 			(effects

Commit message: PCB RevF a3
Connections:
- net DCLK renamed SD_SCK
Changed lines of the file:
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@@
 	(title_block
 		(title "Karabas Pro")
-		(date "2024-05-01")
-		(rev "F")
+		(date "2025-10-10")
+		(rev "F a3")
 	)
 	(junction
@@
 		)
 	)
-	(global_label "DCLK"
+	(global_label "SD_SCK"
 		(shape input)
 		(at 39.37 58.42 180)
@@
 		)
 		(property "Intersheetrefs" "${INTERSHEET_REFS}"
-			(at 32.2009 58.42 0)
+			(at 29.8424 58.42 0)
 			(effects
 				(font
@@
 	)
 	(global_label "DATA0"
-		(shape input)
+		(shape output)
 		(at 39.37 63.5 180)
 		(fields_autoplaced yes)
